File: PinHeck.sch (EAGLE design)
At the start: 344 parts, among them IC1 FT232RL-REEL, IC2 PIC32MX795F512L-80I/PT, IC3 CD74HCT244E, IC4 CD74HCT244E, IC5 ULN2803A, J1 500075-1517, J11 No Load, J2 500075-1517, J3 N/A, J6 161-3507-E, P1 TC33X-2-103E, SW1 101-0134-EV, SW2 101-0134-EV, SW3 101-0134-EV, SW4 0S102011MS2QS1, U1 P8X32A-Q44, U10 74HCT2G04GV,125, U11 74HC165D,652, U12 74HC165D,652, U14 MC74HC08ADG, U15 MC74HC08ADG, U16 MC74HC08ADG, U17 MC74HC08ADG, U18 MC74HC08ADG, U19 MC74HC08ADG, U2 FT230XS-R, U20 TIP107, U21 TIP107, U22 TIP107, U23 TIP107, U24 TIP107, U25 TIP107, U26 TIP107, U27 TIP107, U28 TIP102, U29 TIP102, U3 74HC595D-Q100, U30 TIP102, U31 TIP102, U32 TIP102, U33 TIP102, U34 TIP102, U35 TIP102, U36 WS2801, U37 TIP102, U38 WS2801, U39 LM2937IMP-3.3/NOPB, U4 24LC1025-I/P, U40 TIP102, U41 TIP102, U42 TIP102, U43 TIP102, U44 TIP102, U45 TIP102, U46 TIP102, U47 TIP102, U48 TIP102, U49 TIP102, U5 74HC595D-Q100, U50 TIP102, U51 TIP102, U52 CD74HC123M96, U6 TIP102, U7 TIP102, U8 TIP102, U9 TIP102, X1 FQ7050B-8.000, X2 ECS-65-20-4X

Commit message: Neo Pixel Support and Increased 5V OF DOOM
Parts:
- removed C47: .1uF, PP_Passives:CAPACITOR_NON_POLAR0805
- removed R140, R141, R31, R33: 4.7K, PP_Passives:RESISTOR0805
- removed R25, R26, R27, R28, R29: 10K, PP_Passives:RESISTOR0805
- removed SD1: SD-RSMT-2-MQ, PP_Connectors:SD_CARDSD-RSMT-2-MQ
- removed USBDM, USBDP, VBUS: (no value), PP_Connectors:PH_1X02HEADER_PTH
- added NEO_PIXEL: 26-64-4030, PP_Connectors:PH_1X03KK_3
- BOARD_POWER: value 26-60-4040 -> (none); device PP_Connectors:PH_1X04KK_4 -> PP_Connectors:PH_1X08MOLEX_KK_8
- R24: value 10K -> 360
- SW1, SW2, SW3: value 101-0134-EV -> (none); device PP_Electromechanical:SPST101-0134-EV -> MF_Switches:TACT_6MM
Connections:
- removed net N$16: R29.2, SD1.RW
- new net NEO_DATA: NEO_PIXEL.3, R24.2
- net 3.3V: no longer C47.2, R24.1, R25.1, R26.1, R27.1, R28.1, R29.1, SD1.3.3V
- net 5V: now also BOARD_POWER.6, NEO_PIXEL.1
- net DM: no longer USBDM.2
- net DP: no longer USBDP.2
- net GND: now also BOARD_POWER.5, BOARD_POWER.8, NEO_PIXEL.2, SW1.P$1, SW2.P$2, SW3.P$1, SW3.P$2; no longer C47.1, SD1.GND, SW1.A, SW2.A, SW3.B
- net N$10: now also R24.1; no longer R27.2, SD1.IRQ
- net N$9: now also SW1.P$3; no longer SW1.B
- net P10: no longer R140.1
- net P11: no longer R141.1
- net P12: no longer R31.1
- net P13: no longer R33.1
- net P4: no longer R26.2, SD1.D0
- net P5: no longer R25.2, SD1.SCLK
- net P6: no longer R24.2, SD1.DI
- net P7: no longer R28.2, SD1.CS
- net RES: now also SW2.P$4; no longer SW2.B
- net RG9: now also SW3.P$4; no longer SW3.A
- net S_L: no longer R140.2, R31.2
- net S_R: no longer R141.2, R33.2
- net USBD+: no longer USBDP.1
- net USBD-: no longer USBDM.1
- net USB_BUS: no longer VBUS.2
- net VUSB: no longer VBUS.1
Other:
- moved on the sheet: C46, R24, R32, R34

Commit message: Beefed up 5V line, added caps, added AUX power con.
Parts:
- added AUX_PWR: 26-60-4040, PP_Connectors:PH_1X04KK_4
- added C30: (no value), MF_Passives:CAPACITOR_P_12.5MM
- H1, H18, H2, H3, H4, H5, H6, H7: value MOUNT-HOLE3.2 -> MOUNT-HOLE3.6; device holes:MOUNT-HOLE3.2 -> holes:MOUNT-HOLE3.6
Connections:
- removed net N$10: R24.1
- net 12V: now also AUX_PWR.4
- net 5V: now also AUX_PWR.2, C30.P$1
- net GND: now also AUX_PWR.1, AUX_PWR.3, C30.P$2
- net P4: now also R24.1
