File: Hardware/Pinheck Main Board/PinHeck.sch (EAGLE design)
At the start: 363 parts, among them IC2 PIC32MX795F512L-80I/PT, IC3 CD74HCT244E, IC4 CD74HCT244E, IC5 ULN2803A, J3 N/A, J4 SJ1-2503A, P1 TC33X-2-103E, U1 P8X32A-Q44, U10 74HCT2G04GV,125, U11 CD74HC165M96, U12 CD74HC165M96, U13 CAT24M01LI-G, U14 MC74HC08ADR2G, U15 MC74HC08ADR2G, U16 MC74HC08ADR2G, U17 MC74HC08ADR2G, U18 MC74HC08ADR2G, U19 MC74HC08ADR2G, U2 DS1340Z-33+, U20 TIP107, U21 TIP107, U22 TIP107, U23 TIP107, U24 TIP107, U25 TIP107, U26 TIP107, U27 TIP107, U28 TIP102, U29 TIP102, U3 CD74HC595M96, U30 TIP102, U31 TIP102, U32 TIP102, U33 TIP102, U34 TIP102, U35 TIP102, U36 WS2801, U37 TIP107, U38 WS2801, U39 NCP1117DT33G, U4 CAT24M01LI-G, U40 TIP102, U41 TIP102, U42 TIP102, U43 TIP102, U44 TIP102, U45 TIP102, U46 TIP102, U47 TIP102, U48 TIP102, U49 TIP102, U5 CD74HC595M96, U50 TIP102, U51 TIP102, U52 CD74HC123M96, U6 TIP102, U7 TIP102, U8 TIP102, U9 TIP102, X1 FQ7050B-8.000, X2 9C-6.500MAAJ-T, X3 ABS25-32.768KHz-1-T

Commit message: Routing external connectors first. Working my way inwards.
Parts:
- BOARD_POWER: LABEL01 (none) -> 5V; LABEL02 (none) -> 12V; LABEL03 (none) -> GND
- CABINET: LABEL01 (none) -> GND; LABEL02 (none) -> ST_LI; LABEL03 (none) -> ST_BU; LABEL04 (none) -> TILT; LABEL05 (none) -> COIN; LABEL06 (none) -> ENTER; LABEL07 (none) -> BACK; LABEL08 (none) -> DOOR; LABEL09 (none) -> USER_0; LABEL10 (none) -> R_FLIP; LABEL11 (none) -> L_FLIP
- CAB_RGB: LABEL01 (none) -> 12V; LABEL02 (none) -> 12V; LABEL03 (none) -> BL; LABEL04 (none) -> GL; LABEL05 (none) -> RL; LABEL06 (none) -> BR; LABEL07 (none) -> GR; LABEL08 (none) -> RR; LABEL09 (none) -> GND; LABEL10 (none) -> GND
- LIGHT_COL: LABEL01 (none) -> 12V; LABEL02 (none) -> LIGHT_C_0; LABEL03 (none) -> LIGHT_C_1; LABEL04 (none) -> LIGHT_C_2; LABEL05 (none) -> LIGHT_C_3; LABEL06 (none) -> LIGHT_C_4; LABEL07 (none) -> LIGHT_C_5; LABEL08 (none) -> LIGHT_C_6; LABEL09 (none) -> LIGHT_C_7
- LIGHT_ROW: LABEL01 (none) -> 5V; LABEL02 (none) -> LIGHT_R_0; LABEL03 (none) -> LIGHT_R_1; LABEL04 (none) -> LIGHT_R_2; LABEL05 (none) -> LIGHT_R_3; LABEL06 (none) -> LIGHT_R_4; LABEL07 (none) -> LIGHT_R_5; LABEL08 (none) -> LIGHT_R_6; LABEL09 (none) -> LIGHT_R_7
- SW_COL: LABEL01 (none) -> GND; LABEL02 (none) -> SW_C_7; LABEL03 (none) -> SW_C_6; LABEL04 (none) -> SW_C_5; LABEL05 (none) -> SW_C_4; LABEL06 (none) -> SW_C_3; LABEL07 (none) -> SW_C_2; LABEL08 (none) -> SW_C_1; LABEL09 (none) -> SW_C_0
- SW_ROW: LABEL01 (none) -> GND; LABEL02 (none) -> SW_R_7; LABEL03 (none) -> SW_R_6; LABEL04 (none) -> SW_R_5; LABEL05 (none) -> SW_R_4; LABEL06 (none) -> SW_R_3; LABEL07 (none) -> SW_R_2; LABEL08 (none) -> SW_R_1; LABEL09 (none) -> SW_R_0
- renumbered J4 to AUDIO, J6 to CAB_RGB

Commit message: have all the peripherals layed out on the new pinheck
Parts:
- removed J3: N/A, PP_Connectors:CON_01X04_2.54MM_PIN_HEADER
- added C29: MF-CAP-12.5MM-1000uF, MF_Passives:CAPACITOR_P_6.3MM
- added C30: .1uF, PP_Passives:CAPACITOR_NON_POLAR_0805
- added F5: 4245K, PP_Passives:PTC_FUSE_4245K
- DMD_PWR: LABEL01 (none) -> 12V; LABEL02 (none) -> 5V; LABEL03 (none) -> GND
- GI_0: LABEL01 (none) -> GI_0; LABEL02 (none) -> GI_1; LABEL03 (none) -> GI_2; LABEL04 (none) -> GI_3; LABEL05 (none) -> GI_4; LABEL06 (none) -> GI_5; LABEL07 (none) -> GI_6; LABEL08 (none) -> GI_7; LABEL09 (none) -> 5V
- GI_1: LABEL01 (none) -> GI_8; LABEL02 (none) -> GI_9; LABEL03 (none) -> GI_10; LABEL04 (none) -> GI_11; LABEL05 (none) -> GI_12; LABEL06 (none) -> GI_13; LABEL07 (none) -> GI_14; LABEL08 (none) -> GI_15; LABEL09 (none) -> 5V
- renumbered J7 to DMD_PWR, U40 to GI4, U41 to GI5, U42 to GI6, U43 to GI7, U44 to GI8, U45 to GI9, U46 to GI10, U47 to GI11, U48 to GI12, U49 to GI13, U50 to GI14, U51 to GI15, U6 to GI0, U7 to GI1, U8 to GI2, U9 to GI3
Connections:
- net GI_R_15 renamed GI15
- removed net GI_5V: F4.P$2, GI_0.PIN9, GI_1.PIN9
- new net GI0_5V: F5.P$2, GI_0.PIN9
- new net GI1_5V: F4.P$2, GI_1.PIN9
- net !AN_BLANK: no longer J3.4
- net 12V: now also C29.P$1
- net 5V: now also C30.1, F5.P$1
- net GND: now also C29.P$2, C30.2; no longer J3.2, J3.3
- net WATCHDOG: no longer J3.1
