File: Hardware/Pinheck Main Board/PinHeck.brd (EAGLE design)
At the start: 359.2 x 152.3 mm, 370 parts, among them IC2 PIC32MX795F512L-80I/PT, IC3 CD74HCT244E, IC4 CD74HCT244E, IC5 ULN2803A, P1 TC33X-2-103E, U1 P8X32A-Q44, U10 74HCT2G04GV,125, U11 CD74HC165M96, U12 CD74HC165M96, U13 CAT24M01LI-G, U14 MC74HC08ADR2G, U15 MC74HC08ADR2G, U16 MC74HC08ADR2G, U17 MC74HC08ADR2G, U18 MC74HC08ADR2G, U19 MC74HC08ADR2G, U2 DS1340Z-33+, U20 TIP107, U21 TIP107, U22 TIP107, U23 TIP107, U24 TIP107, U25 TIP107, U26 TIP107, U27 TIP107, U28 TIP102, U29 TIP102, U3 CD74HC595M96, U30 TIP102, U31 TIP102, U32 TIP102, U33 TIP102, U34 TIP102, U35 TIP102, U36 WS2801, U38 WS2801, U39 NCP1117DT33G, U4 CAT24M01LI-G, U5 CD74HC595M96, U52 CD74HC123M96, X1 FQ7050B-8.000, X2 9C-6.500MAAJ-T, X3 ABS25-32.768KHz-1-T

Commit message: Added RGB_COM_OUT_1
Parts:
- removed RGB_COM_OUT: 26-64-4050, PP_Connectors:26-64-4050(KEYPIN2)
- added RGB_COM_OUT_0: 26-64-4050, PP_Connectors:26-64-4050(KEYPIN2)
- added RGB_COM_OUT_1: 26-64-4080, PP_Connectors:26-64-4080(KEYPIN2)
- MOD_CON: device PP_Connectors:2.54MM_01X06_PIN_HEADER -> PP_Connectors:2.54MM_01X08_PIN_HEADER
- OPTO_1, OPTO_2, OPTO_3, OPTO_4, OPTO_5, OPTO_6, OPTO_7: value (none) -> 26-64-4040
- moved U$1 118.3 mm to (236.0, 87.4)
- moved U$2 67.3 mm to (230.9, 74.4)
- moved C19 9.04 mm to (113.0, 120.9), turned to 90 degrees
- moved R13 5.84 mm to (102.6, 83.1)
- moved R14 5.84 mm to (99.8, 83.1)
- moved PICKIT3 4.06 mm to (106.4, 66.3)
- moved PICKIT3_TC 4.06 mm to (99.6, 62.7)
- moved LOGO1 2.65 mm to (95.5, 78.2)
- moved H22 1.02 mm to (99.0, 146.6)
- moved SERVO_0 0.76 mm to (108.0, 147.3)
- moved SERVO_1 0.76 mm to (116.8, 147.3)
- moved SERVO_2 0.76 mm to (108.0, 140.0)
- moved SERVO_3 0.76 mm to (116.8, 140.0)
- moved SERVO_4 0.76 mm to (108.0, 132.6)
- moved GI_1 0.25 mm to (324.1, 6.10)
Connections:
- removed net P4: U1.1
- removed net P5: U1.2
- removed net P6: U1.3
- removed net P7: U1.4
- new net EXT_RGB_CLK_1: RGB_COM_OUT_1.P$3, U1.2
- new net EXT_RGB_DATA_1: RGB_COM_OUT_1.P$2, U1.1
- new net PROP_AUX0: RGB_COM_OUT_1.P$4, U1.3
- new net PROP_AUX1: RGB_COM_OUT_1.P$5, U1.4
- net 12V: now also RGB_COM_OUT_1.P$6
- net 5V: now also RGB_COM_OUT_0.P$4, RGB_COM_OUT_1.P$7; no longer RGB_COM_OUT.P$4
- net EXT_RGB_CLK: now also RGB_COM_OUT_0.P$3; no longer RGB_COM_OUT.P$3
- net EXT_RGB_DATA: now also RGB_COM_OUT_0.P$2; no longer RGB_COM_OUT.P$2
- net GND: now also RGB_COM_OUT_0.P$1, RGB_COM_OUT_1.P$1; no longer RGB_COM_OUT.P$1
- net SERVO_3: now also MOD_CON.7
- net SERVO_4: now also MOD_CON.8
Routing:
- net SERVO_3: track 132.7 -> 236.8 mm, vias 2 -> 4
- net SERVO_4: track 136.2 -> 237.7 mm, vias 2 -> 4
- net EXT_RGB_DATA: track 98.2 -> 116.5 mm
- net EXT_RGB_CLK: track 97.1 -> 110.9 mm
- net SERVO_1: track 122.0 -> 129.1 mm
- net SERVO_0: track 168.3 -> 175.3 mm
- net PIC_LIGHT_C_7: track 239.9 -> 234.1 mm
- net PIC_LIGHT_C_6: track 229.0 -> 223.2 mm
- net SERVO_2: track 153.7 -> 157.0 mm
- net P32_MCLR: track 63.3 -> 65.7 mm
- net N$33: track 24.1 -> 25.8 mm
- net N$31: track 39.4 -> 41.2 mm
- net RX_PROP: track 182.9 -> 184.7 mm
- net 12V: track 597.1 -> 598.6 mm
- net TX_PROP: track 171.6 -> 173.1 mm
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
Commit message: Added more things to PHAM.
Parts:
- removed RGB_COM_OUT_0: 26-64-4050, PP_Connectors:26-64-4050(KEYPIN2)
- removed RGB_COM_OUT_1: 26-64-4080, PP_Connectors:26-64-4080(KEYPIN2)
- added H1, H2: MOUNT_HOLE150MIL, PP_Connectors:MOUNT_HOLE_150MIL
- added RGB_COM_OUT: 26-64-4080, PP_Connectors:26-64-4080(KEYPIN2)
- MOD_CON: device PP_Connectors:2.54MM_01X08_PIN_HEADER -> PP_Connectors:2.54MM_01X20_PIN_HEADER
- moved MOD_CON 15.2 mm to (260.4, 115.1)
- moved R18 14.0 mm to (288.8, 100.1)
- moved R22 14.0 mm to (286.0, 100.1)
- moved H29 13.2 mm to (151.4, 133.6)
- moved R23 7.18 mm to (278.4, 119.1), turned to 0 degrees
- moved R176 2.62 mm to (222.5, 82.3)
- moved C31 0.25 mm to (206.3, 82.8)
- moved C47 0.25 mm to (208.8, 82.8)
- renumbered PROP_PROGRAM to PROP_CONFIG
Connections:
- net P23 renamed PROP_AUX9
- removed net EXT_RGB_CLK_1: RGB_COM_OUT_1.P$3, U1.2
- removed net EXT_RGB_DATA_1: RGB_COM_OUT_1.P$2, U1.1
- removed net P10: U1.11
- removed net P11: U1.12
- removed net P12: U1.13
- removed net P8: U1.9
- removed net P9: U1.10
- new net N$42: MOD_CON.19
- new net N$44: MOD_CON.20
- new net PROP_AUX2: MOD_CON.12, U1.3
- new net PROP_AUX3: MOD_CON.13, U1.4
- new net PROP_AUX4: MOD_CON.14, U1.9
- new net PROP_AUX5: MOD_CON.15, U1.10
- new net PROP_AUX6: MOD_CON.16, U1.11
- new net PROP_AUX7: MOD_CON.17, U1.12
- new net PROP_AUX8: MOD_CON.18, U1.13
- net 12V: now also MOD_CON.7, RGB_COM_OUT.P$6; no longer MOD_CON.6, RGB_COM_OUT_1.P$6
- net 5V: now also RGB_COM_OUT.P$7; no longer RGB_COM_OUT_0.P$4, RGB_COM_OUT_1.P$7
- net EXT_RGB_CLK: now also RGB_COM_OUT.P$5; no longer RGB_COM_OUT_0.P$3
- net EXT_RGB_DATA: now also RGB_COM_OUT.P$4; no longer RGB_COM_OUT_0.P$2
- net GND: now also MOD_CON.11, MOD_CON.6, MOD_CON.8, RGB_COM_OUT.P$1; no longer RGB_COM_OUT_0.P$1, RGB_COM_OUT_1.P$1
- net PROP_AUX0: now also RGB_COM_OUT.P$3, U1.1; no longer RGB_COM_OUT_1.P$4, U1.3
- net PROP_AUX1: now also RGB_COM_OUT.P$2, U1.2; no longer RGB_COM_OUT_1.P$5, U1.4
- net SERVO_3: now also MOD_CON.9; no longer MOD_CON.7
- net SERVO_4: now also MOD_CON.10; no longer MOD_CON.8
Routing:
- net PROP_AUX1: track 0.00 -> 168.9 mm, vias 0 -> 4
- net PROP_AUX0: track 0.00 -> 166.0 mm, vias 0 -> 4
- net PROP_AUX3: track 0.00 -> 94.1 mm, vias 0 -> 2
- net PROP_AUX8: track 0.00 -> 92.1 mm, vias 0 -> 2
- net PROP_AUX7: track 0.00 -> 89.8 mm, vias 0 -> 2
- net PROP_AUX2: track 0.00 -> 89.6 mm, vias 0 -> 2
- net PROP_AUX6: track 0.00 -> 87.9 mm, vias 0 -> 2
- net PROP_AUX5: track 0.00 -> 86.6 mm, vias 0 -> 2
- net PROP_AUX4: track 0.00 -> 85.1 mm, vias 0 -> 2
- net 3.3V: track 243.4 -> 237.4 mm
- net 12V: track 598.6 -> 604.2 mm
- net SD_DO: track 137.1 -> 133.8 mm
- net SERVO_4: track 237.7 -> 240.5 mm
- net RGB_CLK: track 68.3 -> 65.6 mm
- net RGB_DATA: track 74.5 -> 71.8 mm
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
Commit message: Adding fuses.
Parts:
- removed H1, H29: MOUNT_HOLE150MIL, PP_Connectors:MOUNT_HOLE_150MIL
- removed P1: TC33X-2-103E, PP_Passives:TC33_TRIMMER
- added C56, C57: .1uF, PP_Passives:0805
- added F6: 4628, PP_Passives:4628
- added H3, H4: MOUNT_HOLE150MIL, PP_Connectors:MOUNT_HOLE_150MIL
- added R147, R148, R149, R150, R151, R152, R153, R154, R155, R156: 100, PP_Passives:0805
- F1, F2, F3, F4, F5: value 4245K -> 4628; device PP_Passives:4245K -> PP_Passives:4628
- R134: value 20K -> 25K
- U11, U12: value CD74HC165M96 -> 74HC165D-Q100,118
- moved U$1 54.0 mm to (280.9, 57.4)
- moved R18 14.2 mm to (291.6, 114.0)
- moved R22 14.2 mm to (288.8, 114.0)
- moved H11 11.9 mm to (4.57, 16.5)
- moved F1 7.11 mm to (264.9, 37.1)
- moved F2 7.11 mm to (277.1, 37.1)
- moved F3 7.11 mm to (289.3, 37.1)
- moved F4 7.11 mm to (301.5, 37.1)
- moved F5 7.11 mm to (327.7, 37.1)
- moved C19 2.79 mm to (113.0, 118.1)
- moved SW_ROW 2.54 mm to (26.8, 6.10)
- moved H2 1.52 mm to (290.3, 78.0)
- moved C46 1.27 mm to (293.4, 114.0)
- moved H30 1.17 mm to (270.0, 147.7)
- moved H23 1.14 mm to (53.7, 4.57)
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- renumbered MOD_CON to PHABULOUS
Connections:
- removed net N$497: P1.2, R134.1
- new net N$17: CABINET.P$2, R147.1
- new net N$18: CABINET.P$3, R148.1
- new net N$24: CABINET.P$4, R149.1
- new net N$27: CABINET.P$5, R150.1
- new net N$30: CABINET.P$6, R151.1
- new net N$32: CABINET.P$7, R152.1
- new net N$35: CABINET.P$8, R153.1
- new net N$36: CABINET.P$9, R154.1
- new net N$39: CABINET.P$10, R155.1
- new net N$46: CABINET.P$11, R156.1
- new net SERVO_5V: F6.P$2, SERVO_0.P$2, SERVO_1.P$2, SERVO_2.P$2, SERVO_3.P$2, SERVO_4.P$2
- net 3.3V: now also C56.1, C57.1
- net 50V: now also F1.P$1, F2.P$1, F3.P$1; no longer F1.1A, F1.1B, F2.1A, F2.1B, F3.1A, F3.1B
- net 50V_FUSE_0: now also F1.P$2; no longer F1.2A, F1.2B
- net 50V_FUSE_1: now also F2.P$2; no longer F2.2A, F2.2B
- net 50V_FUSE_2: now also F3.P$2; no longer F3.2A, F3.2B
- net 5V: now also F4.P$1, F5.P$1, F6.P$1; no longer F4.1A, F4.1B, F5.1A, F5.1B, SERVO_0.P$2, SERVO_1.P$2, SERVO_2.P$2, SERVO_3.P$2, SERVO_4.P$2
- net BACK: now also R152.2; no longer CABINET.P$7
- net COIN: now also R150.2; no longer CABINET.P$5
- net DOOR: now also R153.2; no longer CABINET.P$8
- net ENTER: now also R151.2; no longer CABINET.P$6
- net GI0_5V: now also F5.P$2; no longer F5.2A, F5.2B
- net GI1_5V: now also F4.P$2; no longer F4.2A, F4.2B
- net GND: now also C56.2, C57.2
- net L_FLIP: now also R156.2; no longer CABINET.P$11
- net R_FLIP: now also R155.2; no longer CABINET.P$10
- net ST_BU: now also R148.2; no longer CABINET.P$3
- net ST_LI: now also R147.2; no longer CABINET.P$2
- net TILT: now also R149.2; no longer CABINET.P$4
- net USER_0: now also R154.2; no longer CABINET.P$9
- net WATCHDOG_ADJUST: now also R134.1; no longer P1.3
Routing:
- net SERVO_5V: track 0.00 -> 41.2 mm
- net GND: track 390.4 -> 417.2 mm
- net CAB_GI_OUT: track 206.3 -> 221.8 mm
- net 3.3V: track 237.4 -> 251.4 mm, vias 105 -> 106
- net N$497: track 13.7 -> 0.00 mm
- net COIN: track 37.4 -> 28.8 mm
- net DOOR: track 20.6 -> 12.1 mm
- net 50V_FUSE_2: track 89.7 -> 81.2 mm
- net 50V_FUSE_1: track 130.2 -> 121.7 mm
- net GI1_5V: track 62.1 -> 53.6 mm
- net R_FLIP: track 20.9 -> 12.5 mm
- net ST_BU: track 25.4 -> 17.0 mm
- net ENTER: track 34.7 -> 26.3 mm
- net TILT: track 39.8 -> 31.4 mm
- net L_FLIP: track 23.0 -> 14.7 mm
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Other:
- board text added: "Pin Heck Addon Board / User Logic Optional Universal Slot. PHABULOUS"

Commit message: TPS chips added and fuses added.
Parts:
- removed C38, C42: EEE-1VA101XP, PP_Passives:6.3MM_CAP_SMD
- removed H20: MOUNT_HOLE150MIL, PP_Connectors:MOUNT_HOLE_150MIL
- added C58, C60: 0.1uF, PP_Passives:0805
- added C59: 2.2nF, PP_Passives:0805
- added C61: 5.6nF, PP_Passives:0805
- added F7: 4628, PP_Passives:4628
- added FLASHER: 26-64-4020, PP_Connectors:26-64-4020
- added R146: 75K, PP_Passives:0805
- added R157: 110K, PP_Passives:0805
- added U6: TPS259251, PP_PowerIC:TPS2592(50/51/60/61)_VSON-10
- added U7: TPS259261, PP_PowerIC:TPS2592(50/51/60/61)_VSON-10
- AUDIO: value SJ1-2503A -> SJ1-3513-SMT; device PP_Connectors:161-3507-E -> PP_Connectors:SJ1-351(3/4/5)-SMT
- CAB_RGB: value (none) -> 26-64-4110
- moved F5 18.8 mm to (327.7, 55.9)
- moved C40 15.8 mm to (28.4, 129.0)
- moved C41 15.8 mm to (28.4, 127.0)
- moved C45 15.6 mm to (19.3, 126.7), turned to 180 degrees
- moved C44 15.6 mm to (19.3, 128.8), turned to 180 degrees
- moved C43 15.5 mm to (19.3, 131.3), turned to 180 degrees
- moved C39 15.5 mm to (28.4, 131.3)
- moved C17 14.5 mm to (20.8, 117.6), turned to 180 degrees
- moved C16 13.9 mm to (34.8, 117.6), turned to 0 degrees
- moved R34 9.70 mm to (321.6, 138.2), turned to 0 degrees
- moved R32 6.90 mm to (312.2, 138.2), turned to 180 degrees
- moved R20 5.04 mm to (298.2, 114.0), turned to 90 degrees
- moved AUDIO 1.30 mm to (316.7, 152.1)
- moved R117 0.76 mm to (34.5, 144.0)
- moved PSU_PWR 0.51 mm to (34.5, 148.3)
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Connections:
- new net 12V_IN: BOARD_POWER.3, C60.1, U7.P$2, U7.P$3, U7.P$4, U7.P$5
- new net 5V_IN: BOARD_POWER.1, C58.1, U6.P$2, U6.P$3, U6.P$4, U6.P$5
- new net FLASH_12V: F7.P$2, FLASHER.P$1
- new net N$48: R146.1, U6.P$10
- new net N$52: C59.1, U6.P$1
- new net N$55: C61.1, U7.P$1
- new net N$59: R157.1, U7.P$10
- net 12V: now also CAB_RGB.P$3, CAB_RGB.P$7, F7.P$1, U7.P$6, U7.P$7, U7.P$8; no longer BOARD_POWER.3, C42.POS, CAB_RGB.P$1, CAB_RGB.P$2, LIGHT_COL.P$1
- net 5V: now also U6.P$6, U6.P$7, U6.P$8; no longer BOARD_POWER.1, C38.POS, LIGHT_ROW.P$1
- net GND: now also C58.2, C59.2, C60.2, C61.2, FLASHER.P$2, R146.2, R157.2, U6.P$9, U6.PAD, U6.PAD2, U6.PAD3, U6.PAD4, U6.PAD5, U6.PAD6, U6.PAD7, U7.P$9, U7.PAD, U7.PAD2, U7.PAD3, U7.PAD4, U7.PAD5, U7.PAD6, U7.PAD7; no longer C38.NEG, C42.NEG, CAB_RGB.P$10, CAB_RGB.P$9, SW_COL.P$1, SW_ROW.P$1
- net RGB_BOUT_L: now also CAB_RGB.P$4; no longer CAB_RGB.P$3
- net RGB_BOUT_R: now also CAB_RGB.P$8; no longer CAB_RGB.P$6
- net RGB_GOUT_L: now also CAB_RGB.P$5; no longer CAB_RGB.P$4
- net RGB_GOUT_R: now also CAB_RGB.P$9; no longer CAB_RGB.P$7
- net RGB_ROUT_L: now also CAB_RGB.P$6; no longer CAB_RGB.P$5
- net RGB_ROUT_R: now also CAB_RGB.P$10; no longer CAB_RGB.P$8
- net S_L: now also AUDIO.2; no longer AUDIO.5
- net S_R: now also AUDIO.3; no longer AUDIO.2
Routing:
- net 12V: track 604.8 -> 658.2 mm, vias 13 -> 17
- net 5V: track 169.6 -> 131.7 mm, vias 30 -> 41
- net FLASH_12V: track 0.00 -> 27.4 mm
- net GI0_5V: track 45.1 -> 27.5 mm
- net S_L: track 15.3 -> 4.73 mm
- net AUD1: track 154.9 -> 165.1 mm
- net 5V_IN: track 0.00 -> 9.76 mm
- net GND: track 417.2 -> 426.1 mm, vias 147 -> 165
- net AUD0: track 154.0 -> 161.7 mm
- net S_R: track 12.0 -> 5.03 mm
- net RGB_BOUT_L: track 18.9 -> 25.8 mm
- net RGB_BOUT_R: track 15.8 -> 22.6 mm
- net RGB_GOUT_L: track 17.9 -> 23.4 mm
- net RGB_GOUT_R: track 15.8 -> 20.2 mm
- net RGB_ROUT_L: track 16.9 -> 21.0 mm
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- added copper zone on layer 1, net 12V
- added copper zone on layer 16, net 12V
- added copper zone on layer 1, net 12V_IN
- added copper zone on layer 1, net 5V
- added copper zone on layer 1, net 5V_IN
- added copper zone on layer 16, net GND
Other:
- outline, holes or cut-outs redrawn

Commit message: started edge con routing.
Parts:
- added D3: SMBJ6.0CA, PP_Passives:SMBJ
- added D4: SMBJ15CA, PP_Passives:SMBJ
- added J1: N/A, PP_Connectors:2.54MM_01X04_PIN_HEADER
- moved DMD_CON 6.18 mm to (263.1, 126.0)
- moved R21 4.67 mm to (305.8, 114.0), turned to 90 degrees
- moved C59 2.95 mm to (34.4, 135.0)
- moved C16 2.03 mm to (34.8, 115.6)
- moved C17 2.03 mm to (20.8, 115.6)
- moved C39 2.03 mm to (28.4, 129.3)
- moved C40 2.03 mm to (28.4, 127.0)
- moved C43 2.03 mm to (19.3, 129.3)
- moved C58 2.03 mm to (27.9, 134.1)
- moved C60 2.03 mm to (18.8, 134.1)
- moved C61 2.03 mm to (24.9, 135.9)
- moved R146 2.03 mm to (32.8, 130.0)
- moved R157 2.03 mm to (23.6, 130.0)
- moved C41 2.03 mm to (28.4, 125.0)
- moved C44 2.03 mm to (19.3, 126.7)
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Connections:
- removed net N$42: PHABULOUS.19
- new net N$100: J12.P$88
- new net N$101: J12.P$89
- new net N$102: J12.P$90
- new net N$103: J12.P$101
- new net N$104: J12.P$103
- new net N$105: J12.P$105
- new net N$106: J12.P$107
- new net N$107: J12.P$109
- new net N$108: J12.P$111
- new net N$109: J12.P$113
- new net N$110: J12.P$115
- new net N$111: J12.P$117
- new net N$112: J12.P$119
- new net N$128: J12.P$8
- new net N$129: J12.P$10
- new net N$130: J12.P$12
- new net N$131: J12.P$14
- new net N$132: J12.P$16
- new net N$133: J12.P$18
- new net N$134: J12.P$20
- new net N$135: J12.P$22
- new net N$136: J12.P$24
- new net N$137: J12.P$26
- new net N$138: J12.P$28
- new net N$139: J12.P$30
- new net N$140: J12.P$32
- new net N$141: J12.P$34
- new net N$142: J12.P$36
- new net N$143: J12.P$38
- new net N$144: J12.P$40
- new net N$145: J12.P$60
- new net N$146: J12.P$59
- new net N$147: J12.P$58
- new net N$148: J12.P$57
- new net N$149: J12.P$56
- new net N$150: J12.P$55
- new net N$151: J12.P$54
- new net N$152: J12.P$53
- new net N$153: J12.P$52
- new net N$154: J12.P$51
- new net N$155: J12.P$62
- new net N$156: J12.P$64
- new net N$157: J12.P$66
- new net N$158: J12.P$68
- new net N$159: J12.P$70
- new net N$160: J12.P$72
- new net N$161: J12.P$74
- new net N$162: J12.P$76
- new net N$163: J12.P$78
- new net N$164: J12.P$80
- new net N$165: J12.P$100
- new net N$166: J12.P$99
- new net N$167: J12.P$98
- new net N$168: J12.P$97
- new net N$169: J12.P$96
- new net N$170: J12.P$95
- new net N$171: J12.P$94
- new net N$172: J12.P$93
- new net N$173: J12.P$92
- new net N$174: J12.P$91
- new net N$175: J12.P$102
- new net N$176: J12.P$104
- new net N$177: J12.P$106
- new net N$178: J12.P$108
- new net N$179: J12.P$110
- new net N$180: J12.P$112
- new net N$181: J12.P$114
- new net N$182: J12.P$116
- new net N$183: J12.P$118
- new net N$184: J12.P$120
- new net N$54: J12.P$7
- new net N$56: J12.P$9
- new net N$57: J12.P$11
- new net N$58: J12.P$13
- new net N$60: J12.P$15
- new net N$61: J12.P$17
- new net N$62: J12.P$19
- new net N$63: J12.P$21
- new net N$64: J12.P$23
- new net N$65: J12.P$25
- new net N$66: J12.P$27
- new net N$67: J12.P$29
- new net N$68: J12.P$31
- new net N$69: J12.P$33
- new net N$70: J12.P$35
- new net N$71: J12.P$37
- new net N$72: J12.P$39
- new net N$73: J12.P$41
- new net N$74: J12.P$42
- new net N$75: J12.P$43
- new net N$76: J12.P$44
- new net N$77: J12.P$45
- new net N$78: J12.P$46
- new net N$79: J12.P$47
- new net N$80: J12.P$48
- new net N$81: J12.P$49
- new net N$82: J12.P$50
- new net N$83: J12.P$61
- new net N$84: J12.P$63
- new net N$85: J12.P$65
- new net N$86: J12.P$67
- new net N$87: J12.P$69
- new net N$88: J12.P$71
- new net N$89: J12.P$73
- new net N$90: J12.P$75
- new net N$91: J12.P$77
- new net N$92: J12.P$79
- new net N$93: J12.P$81
- new net N$94: J12.P$82
- new net N$95: J12.P$83
- new net N$96: J12.P$84
- new net N$97: J12.P$85
- new net N$98: J12.P$86
- new net N$99: J12.P$87
- net 12V_IN: now also D4.CATH
- net 5V_IN: now also D3.CATH
- net AUD0: now also J12.P$5
- net AUD1: now also J12.P$6
- net GND: now also D3.ANODE, D4.ANODE, J1.4
- net PROP_AUX9: now also PHABULOUS.19
- net SD_CS: now also J12.P$1
- net SD_DI: now also J12.P$2
- net SD_DO: now also J12.P$4
- net SD_SCLK: now also J12.P$3
- net USBD+: now also J1.3
- net USBD-: now also J1.2
- net VUSB: now also J1.1
Routing:
- net AUD1: track 165.1 -> 270.6 mm, vias 0 -> 2
- net AUD0: track 161.7 -> 266.2 mm, vias 0 -> 2
- net PROP_AUX9: track 0.00 -> 87.9 mm, vias 0 -> 1
- net SD_DO: track 132.7 -> 191.6 mm, vias 2 -> 4
- net SD_SCLK: track 130.6 -> 185.9 mm, vias 2 -> 4
- net SD_DI: track 125.6 -> 175.6 mm, vias 2 -> 4
- net SD_CS: track 123.8 -> 172.2 mm, vias 2 -> 4
- net 12V: track 658.2 -> 687.1 mm
- net USBD+: track 0.00 -> 26.7 mm
- net USBD-: track 0.00 -> 25.8 mm
- net VUSB: track 0.00 -> 25.4 mm
- net PIC_SOL_3: track 143.9 -> 140.9 mm
- net TX_PIC32: track 92.3 -> 90.2 mm
- net RX_PIC32: track 106.1 -> 103.9 mm
- net GND: track 426.1 -> 428.2 mm
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
Commit message: more routing!
Parts:
- removed R147: 100, PP_Passives:0805
Connections:
- removed net N$128: J12.P$8
- removed net N$129: J12.P$10
- removed net N$130: J12.P$12
- removed net N$131: J12.P$14
- removed net N$132: J12.P$16
- removed net N$17: CABINET.P$2, R147.1
- removed net N$18: CABINET.P$3, R148.1
- removed net N$24: CABINET.P$4, R149.1
- removed net N$27: CABINET.P$5, R150.1
- removed net N$30: CABINET.P$6, R151.1
- removed net N$32: CABINET.P$7, R152.1
- removed net N$35: CABINET.P$8, R153.1
- removed net N$36: CABINET.P$9, R154.1
- removed net N$39: CABINET.P$10, R155.1
- removed net N$46: CABINET.P$11, R156.1
- removed net N$54: J12.P$7
- removed net N$56: J12.P$9
- removed net N$57: J12.P$11
- removed net N$58: J12.P$13
- removed net N$60: J12.P$15
- removed net N$61: J12.P$17
- new net BACK_OUT: CABINET.P$7, J12.P$11, R152.1
- new net COIN_OUT: CABINET.P$5, J12.P$13, R150.1
- new net DOOR_OUT: CABINET.P$8, J12.P$10, R153.1
- new net ENTER_OUT: CABINET.P$6, J12.P$12, R151.1
- new net L_FLIP_OUT: CABINET.P$11, J12.P$7, R156.1
- new net R_FLIP_OUT: CABINET.P$10, J12.P$8, R155.1
- new net ST_BU_OUT: CABINET.P$3, J12.P$15, R148.1
- new net TILT_OUT: CABINET.P$4, J12.P$14, R149.1
- new net USER_0_OUT: CABINET.P$9, J12.P$9, R154.1
- net GI_R_6: now also J12.P$17
- net GI_R_7: now also J12.P$16
- net ST_LI: now also CABINET.P$2; no longer R147.2
Routing:
- net GI_R_6: track 22.4 -> 204.1 mm, vias 0 -> 1
- net GI_R_7: track 24.8 -> 197.6 mm, vias 0 -> 1
- net ST_BU_OUT: track 0.00 -> 149.3 mm, vias 0 -> 1
- net TILT_OUT: track 0.00 -> 143.9 mm, vias 0 -> 1
- net COIN_OUT: track 0.00 -> 140.9 mm, vias 0 -> 1
- net USER_0_OUT: track 0.00 -> 139.9 mm, vias 0 -> 1
- net L_FLIP_OUT: track 0.00 -> 139.3 mm, vias 0 -> 1
- net R_FLIP_OUT: track 0.00 -> 138.8 mm, vias 0 -> 1
- net DOOR_OUT: track 0.00 -> 138.4 mm, vias 0 -> 1
- net BACK_OUT: track 0.00 -> 137.9 mm, vias 0 -> 1
- net ENTER_OUT: track 0.00 -> 137.2 mm, vias 0 -> 1
- net ST_LI: track 16.7 -> 25.4 mm
- net N$17: track 6.89 -> 0.00 mm
- net N$18: track 6.85 -> 0.00 mm
- net N$30: track 6.82 -> 0.00 mm
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