File: Hardware/Pinheck Test Jig/PinHeck Test Jig.brd (EAGLE design)
At the start: 359.2 x 152.3 mm, 194 parts, among them SW1 MF-SW-TACT-6MM, U1 P8X32A-Q44, U2 CAT24C512WI-GT3, U3 FT230XS, U4 IP4234CZ6, U5 NCP1117DT33G, U6 NCP1117DT50G, X1 ABMM-6.000MHZ-B2-T

Commit message: Added AUX, and RGB LED Board. Working on Test Jib.
Parts:
- removed R1, R2: 10K, MF_Passives:R0805
- removed SD1: (no value), PP_Connectors:SD-RSMT-2-MQ
- added C21, C22, C23, C24: 0.1uF, PP_Passives:0805
- added R14, R15: RL73H2BR10FTD, PP_Passives:1206
- added R16, R17: ERJ-6ENF3002V, PP_Passives:0805
- added R18, R19, R20, R21: 10K, PP_Passives:0805
- added TVS1: V18AUMLA2220H, PP_Passives:2220
- added U10, U11: BSO080P03NS3E G, PP_DiscreteSemi:DSO-8
- added U12, U13: MF-DSC-SOT233-MMBT3904, PP_DiscreteSemi:SOT-23-3
- added U14, U15: CD74HC595M96, PP_DigitalIC:CD74HC595_SOIC-16
- added U16, U17, U18, U19, U20, U21, U22, U23, U24, U25, U26, U27, U28, U29, U30, U31: CD74HC165M96, PP_DigitalIC:CD74HC165_SOIC-16
- added U7, U8: INA139NA/3K, PP_AnalogIC:INA169NA/250_SOT-23-5
- added U9: MAX11613EUA+, PP_AnalogIC:MAX11613_UMAX-8
- C1: value 1uF -> 0.1uF; device MF_Passives:C0805 -> PP_Passives:0805
- moved C1 542.0 mm to (-192.3, -148.1), turned to 0 degrees
Connections:
- net IN_OPTO_0 renamed P27
- net IN_OPTO_1 renamed P26
- net IN_OPTO_2 renamed P25
- net IN_OPTO_3 renamed P24
- net IN_OPTO_4 renamed P23
- net IN_OPTO_5 renamed P22
- net IN_OPTO_6 renamed P21
- net IN_OPTO_7 renamed P20
- net LCD_RES renamed P19
- net OUT_OPTO_0 renamed P18
- net OUT_OPTO_1 renamed P17
- net OUT_OPTO_10 renamed P8
- net OUT_OPTO_11 renamed P7
- net OUT_OPTO_12 renamed P6
- net OUT_OPTO_13 renamed P5
- net OUT_OPTO_14 renamed P4
- net OUT_OPTO_15 renamed P3
- net OUT_OPTO_16 renamed P2
- net OUT_OPTO_17 renamed P1
- net OUT_OPTO_2 renamed P16
- net OUT_OPTO_3 renamed P15
- net OUT_OPTO_4 renamed P14
- net OUT_OPTO_5 renamed P13
- net OUT_OPTO_6 renamed P12
- net OUT_OPTO_7 renamed P11
- net OUT_OPTO_8 renamed P10
- net OUT_OPTO_9 renamed P9
- removed net 12V_IN: 12V.P$1
- removed net 5V_IN: 5V.P$1
- new net 12.0V_SW: 12V.P$1, U10.1, U10.2, U10.3
- new net 165_CLK: U16.2, U17.2, U18.2, U19.2, U20.2, U21.2, U22.2, U23.2, U24.2, U25.2, U26.2, U27.2, U28.2, U29.2, U30.2, U31.2
- new net 165_DATA: U16.9
- new net 165_LOAD: U16.1, U17.1, U18.1, U19.1, U20.1, U21.1, U22.1, U23.1, U24.1, U25.1, U26.1, U27.1, U28.1, U29.1, U30.1, U31.1
- new net 5.0V_CUR: R15.2, R20.1, U11.5, U11.6, U11.7, U11.8, U8.4
- new net 5.0V_SW: 5V.P$1, U11.1, U11.2, U11.3
- new net 595_CLK: U14.11, U15.11
- new net 595_DATA: U14.14
- new net 595_LAT: U14.12, U15.12
- new net A_0: C21.1, R16.2, U7.1, U9.P$1
- new net A_1: C22.1, R17.2, U8.1, U9.P$2
- new net N$11: R18.2, U10.4, U12.3
- new net N$12: R20.2, U11.4, U13.3
- new net N$13: R19.2, U12.1
- new net N$14: U20.10, U21.9
- new net N$15: R21.2, U13.1
- new net N$16: U21.10, U22.9
- new net N$17: U22.10, U23.9
- new net N$18: U23.10, U24.9
- new net N$19: U24.10, U25.9
- new net N$20: U16.6
- new net N$21: U14.9, U15.14
- new net N$22: U16.10, U17.9
- new net N$23: U25.10, U26.9
- new net N$24: U17.10, U18.9
- new net N$25: U26.10, U27.9
- new net N$26: U27.10, U28.9
- new net N$27: U28.10, U29.9
- new net N$28: U29.10, U30.9
- new net N$29: U30.10, U31.9
- new net PWR_ON: R19.1, R21.1, U1.41
- new net VIN_CUR: R14.2, R18.1, U10.5, U10.6, U10.7, U10.8, U7.4
- net 3.3V: now also C1.1, C23.1, C24.1, U14.10, U14.16, U15.10, U15.16, U16.16, U17.16, U18.16, U19.16, U20.16, U21.16, U22.16, U23.16, U24.16, U25.16, U26.16, U27.16, U28.16, U29.16, U30.16, U31.16, U7.5, U8.5, U9.P$8; no longer C1.P$2, R1.P$1, R2.P$1, SD1.4
- net 5.0V: now also R15.1, U8.3
- net BACK_OUT: now also U14.4
- net COIN_OUT: now also U14.6
- net DMD_1: now also U29.13
- net DMD_11: now also U29.6
- net DMD_13: now also U30.11
- net DMD_3: now also U29.14
- net DMD_5: now also U29.3
- net DMD_7: now also U29.4
- net DMD_9: now also U29.5
- net DOOR_OUT: now also U14.3
- net ENTER_OUT: now also U14.5
- net EXT_RGB_CLK: now also U28.11
- net EXT_RGB_DATA: now also U28.12
- net GI15: now also U18.11
- net GI_R_0: now also U17.6
- net GI_R_1: now also U17.5
- net GI_R_10: now also U18.4
- net GI_R_11: now also U18.3
- net GI_R_12: now also U18.14
- net GI_R_13: now also U18.13
- net GI_R_14: now also U18.12
- net GI_R_2: now also U17.4
- net GI_R_3: now also U17.3
- net GI_R_4: now also U17.14
- net GI_R_5: now also U17.13
- net GI_R_6: now also U17.12
- net GI_R_7: now also U17.11
- net GI_R_8: now also U18.6
- net GI_R_9: now also U18.5
- net GND: now also C1.2, C21.2, C22.2, C23.2, C24.2, R16.1, R17.1, TVS1.P$2, U12.2, U13.2, U14.13, U14.8, U15.13, U15.8, U16.15, U16.8, U17.15, U17.8, U18.15, U18.8, U19.15, U19.8, U20.15, U20.8, U21.15, U21.8, U22.15, U22.8, U23.15, U23.8, U24.15, U24.8, U25.15, U25.8, U26.15, U26.8, U27.15, U27.8, U28.15, U28.8, U29.15, U29.8, U30.15, U30.8, U31.15, U31.8, U7.2, U8.2, U9.P$7; no longer C1.P$1, SD1.3, SD1.6, SD1.GND_1, SD1.GND_2
- net LIGHT_C_0: now also U24.6, U25.6
- net LIGHT_C_1: now also U24.5, U25.5
- net LIGHT_C_2: now also U24.4, U25.4
- net LIGHT_C_3: now also U24.3, U25.3
- net LIGHT_C_4: now also U24.14, U25.14
- net LIGHT_C_5: now also U24.13, U25.13
- net LIGHT_C_6: now also U24.12, U25.12
- net LIGHT_C_7: now also U24.11, U25.11
- net LIGHT_R_0: now also U23.6
- net LIGHT_R_1: now also U23.5
- net LIGHT_R_2: now also U23.4
- net LIGHT_R_3: now also U23.3
- net LIGHT_R_4: now also U23.14
- net LIGHT_R_5: now also U23.13
- net LIGHT_R_6: now also U23.12
- net LIGHT_R_7: now also U23.11
- net L_FLIP_OUT: now also U14.15
- net N$1: now also U18.10, U19.9; no longer R1.P$2, SD1.9
- net N$2: now also U19.10, U20.9; no longer R2.P$2, SD1.8
- net OPTO_1: now also U26.11
- net OPTO_2: now also U26.12
- net OPTO_3: now also U26.13
- net OPTO_4: now also U26.14
- net OPTO_5: now also U26.3
- net OPTO_6: now also U26.4
- net OPTO_7: now also U26.5
- net PROP_AUX0: now also U28.13
- net PROP_AUX1: now also U28.14
- net RGB_BOUT_L: now also U29.12
- net RGB_BOUT_R: now also U28.5
- net RGB_GOUT_L: now also U29.11
- net RGB_GOUT_R: now also U28.4
- net RGB_ROUT_L: now also U28.6
- net RGB_ROUT_R: now also U28.3
- net R_FLIP_OUT: now also U14.1
- net SCL: now also U9.P$5
- net SDA: now also U9.P$6
- net SD_CS: now also U16.11; no longer SD1.1
- net SD_DI: now also U16.12; no longer SD1.2
- net SD_DO: now also U16.14; no longer SD1.7
- net SD_SCLK: now also U16.13; no longer SD1.5
- net SERVO_0: now also U27.11
- net SERVO_1: now also U27.12
- net SERVO_2: now also U27.13
- net SERVO_3: now also U27.14
- net SERVO_4: now also U27.3
- net SOL_PWR_0: now also U21.6
- net SOL_PWR_1: now also U21.5
- net SOL_PWR_10: now also U20.4
- net SOL_PWR_11: now also U20.3
- net SOL_PWR_12: now also U20.14
- net SOL_PWR_13: now also U20.13
- net SOL_PWR_14: now also U20.12
- net SOL_PWR_15: now also U20.11
- net SOL_PWR_16: now also U19.6
- net SOL_PWR_17: now also U19.5
- net SOL_PWR_18: now also U19.4
- net SOL_PWR_19: now also U19.3
- net SOL_PWR_2: now also U21.4
- net SOL_PWR_20: now also U19.14
- net SOL_PWR_21: now also U19.13
- net SOL_PWR_22: now also U19.12
- net SOL_PWR_23: now also U19.11
- net SOL_PWR_3: now also U21.3
- net SOL_PWR_4: now also U21.14
- net SOL_PWR_5: now also U21.13
- net SOL_PWR_6: now also U21.12
- net SOL_PWR_7: now also U21.11
- net SOL_PWR_8: now also U20.6
- net SOL_PWR_9: now also U20.5
- net ST_LI: now also U16.5
- net SW_C_0: now also U22.11, U31.11
- net SW_C_1: now also U22.12, U30.12, U31.12
- net SW_C_2: now also U22.13, U30.13, U31.13
- net SW_C_3: now also U22.14, U30.14, U31.14
- net SW_C_4: now also U22.3, U30.3, U31.3
- net SW_C_5: now also U22.4, U30.4, U31.4
- net SW_C_6: now also U22.5, U30.5, U31.5
- net SW_C_7: now also U22.6, U30.6, U31.6
- net SW_R_0: now also U15.15
- net SW_R_1: now also U15.1
- net SW_R_2: now also U15.2
- net SW_R_3: now also U15.3
- net SW_R_4: now also U15.4
- net SW_R_5: now also U15.5
- net SW_R_6: now also U15.6
- net SW_R_7: now also U15.7
- net S_L: now also U16.3
- net S_R: now also U16.4
- net TILT_OUT: now also U14.7
- net USB_!RST: no longer U1.41
- net USER_0_OUT: now also U14.2
- net VIN: now also R14.1, TVS1.P$1, U7.3

Commit message: Jig Schematic Done.
Parts:
- removed PIC32_UART, PICKIT3, PROP_UART: (no value), PP_Connectors:2.54MM_01X06_PIN_HEADER
- removed U25, U31: CD74HC165M96, PP_DigitalIC:CD74HC165_SOIC-16
- added !MCLR!/VPP, !RES!_PROP, !RST!_PIC32, ICSPCLK, ICSPDAT, PGM, RX_PIC32, RX_PROP, TX_PIC32, TX_PROP, VDD, VSS: (no value), PP_Connectors:0914-3-15-20-77-14-11-0
- added R1, R100, R2, R22, R23, R24, R25, R26, R27, R28, R29, R31, R32, R33, R34, R35, R36, R37, R38, R39, R40, R41, R42, R43, R44, R45, R46, R47, R48, R49, R50, R51, R52, R53, R54, R55, R56, R57, R58, R59, R60, R61, R62, R63, R64, R65, R66, R67, R68, R69, R70, R71, R72, R73, R74, R75, R76, R77, R78, R79, R80, R81, R82, R83, R84, R93, R94, R97, R98, R99: 10K, MF_Passives:R0603
- added R85, R86, R87, R88, R89, R90, R91, R92: 30K, MF_Passives:R0603
Connections:
- removed net N$19: U24.10, U25.9
- removed net N$20: U16.6
- removed net P1: U1.42
- removed net P10: U1.11
- removed net P11: U1.12
- removed net P12: U1.13
- removed net P2: U1.43
- removed net P3: U1.44
- removed net P4: U1.1
- removed net P5: U1.2
- removed net P6: U1.3
- removed net P7: U1.4
- removed net P8: U1.9
- removed net P9: U1.10
- removed net SOL_GND: SOL_GND.P$1
- new net !RES!_PROP: !RES!_PROP.P$1, U1.13
- new net !RST!_PIC32: !RST!_PIC32.P$1, U1.10
- new net N$30: !MCLR!/VPP.P$1, PICKIT3_IN.1
- new net N$31: PICKIT3_IN.2, VDD.P$1
- new net N$33: PICKIT3_IN.3, VSS.P$1
- new net N$34: ICSPDAT.P$1, PICKIT3_IN.4
- new net N$35: ICSPCLK.P$1, PICKIT3_IN.5
- new net N$36: PGM.P$1, PICKIT3_IN.6
- new net N$37: R83.P$2, R91.P$1, U24.12
- new net N$38: R82.P$2, R90.P$1, U24.13
- new net N$39: R81.P$2, R89.P$1, U24.14
- new net N$40: R80.P$2, R88.P$1, U24.3
- new net N$41: R79.P$2, R87.P$1, U24.4
- new net N$42: R78.P$2, R86.P$1, U24.5
- new net N$43: R77.P$2, R85.P$1, U24.6
- new net RX_PIC32: RX_PIC32.P$1, U1.4
- new net RX_PROP: RX_PROP.P$1, U1.11
- new net TX_PIC32: TX_PIC32.P$1, U1.9
- new net TX_PROP: TX_PROP.P$1, U1.12
- net 165_CLK: now also U1.1; no longer U25.2, U31.2
- net 165_DATA: now also U1.3
- net 165_LOAD: now also U1.2; no longer U25.1, U31.1
- net 3.3V: now also R1.P$1, R100.P$1, R2.P$1, R22.P$1, R23.P$1, R24.P$1, R25.P$1, R26.P$1, R27.P$1, R28.P$1, R29.P$1, R31.P$1, R32.P$1, R33.P$1, R34.P$1, R35.P$1, R36.P$1, R37.P$1, R38.P$1, R39.P$1, R40.P$1, R41.P$1, R42.P$1, R43.P$1, R44.P$1, R45.P$1, R46.P$1, R47.P$1, R48.P$1, R49.P$1, R50.P$1, R51.P$1, R52.P$1, R53.P$1, R54.P$1, R55.P$1, R56.P$1, R57.P$1, R58.P$1, R59.P$1, R60.P$1, R61.P$1, R62.P$1, R63.P$1, R64.P$1, R65.P$1, R66.P$1, R67.P$1, R68.P$1, R69.P$1, R70.P$1, R71.P$1, R72.P$1, R73.P$1, R74.P$1, R75.P$1, R76.P$1, R93.P$1, R94.P$1, R97.P$1, R98.P$1, R99.P$1; no longer U25.16, U31.16
- net 595_CLK: now also U1.42
- net 595_DATA: now also U1.44
- net 595_LAT: now also U1.43
- net GI15: now also R28.P$2
- net GI_R_0: now also R27.P$2
- net GI_R_1: now also R26.P$2
- net GI_R_10: now also R34.P$2
- net GI_R_11: now also R33.P$2
- net GI_R_12: now also R32.P$2
- net GI_R_13: now also R31.P$2
- net GI_R_14: now also R29.P$2
- net GI_R_2: now also R25.P$2
- net GI_R_3: now also R24.P$2
- net GI_R_4: now also R23.P$2
- net GI_R_5: now also R22.P$2
- net GI_R_6: now also R2.P$2
- net GI_R_7: now also R1.P$2
- net GI_R_8: now also R36.P$2
- net GI_R_9: now also R35.P$2
- net GND: now also R77.P$1, R78.P$1, R79.P$1, R80.P$1, R81.P$1, R82.P$1, R83.P$1, R84.P$1, SOL_GND.P$1; no longer U25.15, U25.8, U31.15, U31.8
- net LIGHT_C_0: now also R85.P$2; no longer U24.6, U25.6
- net LIGHT_C_1: now also R86.P$2; no longer U24.5, U25.5
- net LIGHT_C_2: now also R87.P$2; no longer U24.4, U25.4
- net LIGHT_C_3: now also R88.P$2; no longer U24.3, U25.3
- net LIGHT_C_4: now also R89.P$2; no longer U24.14, U25.14
- net LIGHT_C_5: now also R90.P$2; no longer U24.13, U25.13
- net LIGHT_C_6: now also R91.P$2; no longer U24.12, U25.12
- net LIGHT_C_7: now also R92.P$2; no longer U24.11, U25.11
- net LIGHT_R_0: now also R76.P$2
- net LIGHT_R_1: now also R75.P$2
- net LIGHT_R_2: now also R74.P$2
- net LIGHT_R_3: now also R73.P$2
- net LIGHT_R_4: now also R72.P$2
- net LIGHT_R_5: now also R71.P$2
- net LIGHT_R_6: now also R70.P$2
- net LIGHT_R_7: now also R69.P$2
- net N$23: now also U24.10; no longer U25.10
- net N$29: now also R84.P$2, R92.P$1, U24.11; no longer U30.10, U31.9
- net RGB_BOUT_L: now also R94.P$2
- net RGB_BOUT_R: now also R99.P$2
- net RGB_GOUT_L: now also R93.P$2
- net RGB_GOUT_R: now also R98.P$2
- net RGB_ROUT_L: now also R100.P$2
- net RGB_ROUT_R: now also R97.P$2
- net SOL_PWR_0: now also R60.P$2
- net SOL_PWR_1: now also R59.P$2
- net SOL_PWR_10: now also R50.P$2
- net SOL_PWR_11: now also R49.P$2
- net SOL_PWR_12: now also R48.P$2
- net SOL_PWR_13: now also R47.P$2
- net SOL_PWR_14: now also R46.P$2
- net SOL_PWR_15: now also R45.P$2
- net SOL_PWR_16: now also R44.P$2
- net SOL_PWR_17: now also R43.P$2
- net SOL_PWR_18: now also R42.P$2
- net SOL_PWR_19: now also R41.P$2
- net SOL_PWR_2: now also R58.P$2
- net SOL_PWR_20: now also R40.P$2
- net SOL_PWR_21: now also R39.P$2
- net SOL_PWR_22: now also R38.P$2
- net SOL_PWR_23: now also R37.P$2
- net SOL_PWR_3: now also R57.P$2
- net SOL_PWR_4: now also R56.P$2
- net SOL_PWR_5: now also R55.P$2
- net SOL_PWR_6: now also R54.P$2
- net SOL_PWR_7: now also R53.P$2
- net SOL_PWR_8: now also R52.P$2
- net SOL_PWR_9: now also R51.P$2
- net SW_C_0: now also R61.P$2; no longer U31.11
- net SW_C_1: now also R62.P$2; no longer U30.12, U31.12
- net SW_C_2: now also R63.P$2; no longer U30.13, U31.13
- net SW_C_3: now also R64.P$2; no longer U30.14, U31.14
- net SW_C_4: now also R65.P$2; no longer U30.3, U31.3
- net SW_C_5: now also R66.P$2; no longer U30.4, U31.4
- net SW_C_6: now also R67.P$2; no longer U30.5, U31.5
- net SW_C_7: now also R68.P$2; no longer U30.6, U31.6

Commit message: Routing Test Jig.
Parts:
- removed SW1: MF-SW-TACT-6MM, MF_Switches:TACT6MM
- added C25: 0.1uF, MF_Passives:C0603
- moved R94 844.9 mm to (354.8, 164.8), turned to 90 degrees
- moved R93 844.5 mm to (354.8, 161.4), turned to 90 degrees
- moved R99 830.9 mm to (344.9, 164.8), turned to 90 degrees
- moved R98 830.5 mm to (344.9, 161.4), turned to 90 degrees
- moved R97 826.2 mm to (341.6, 164.8), turned to 90 degrees
- moved R100 816.6 mm to (335.0, 161.4), turned to 90 degrees
- moved R92 812.3 mm to (331.7, 164.8), turned to 90 degrees
- moved R91 811.9 mm to (331.7, 161.4), turned to 90 degrees
- moved R90 807.6 mm to (328.4, 164.8), turned to 90 degrees
- moved R89 807.2 mm to (328.4, 161.4), turned to 90 degrees
- moved R88 802.9 mm to (325.1, 164.8), turned to 90 degrees
- moved R87 802.6 mm to (325.1, 161.4), turned to 90 degrees
- moved R86 798.3 mm to (321.8, 164.8), turned to 90 degrees
- moved R85 797.9 mm to (321.8, 161.4), turned to 90 degrees
- moved R84 793.6 mm to (318.5, 164.8), turned to 90 degrees
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Connections:
- removed net N$7: C9.P$2, R6.P$1, SW1.P$3
- net 3.3V: now also C25.P$1
- net GND: now also C25.P$2
- net PROP_!RST: now also C9.P$2, R6.P$1; no longer SW1.P$2
Routing:
- net PROP_!RST: track 0.00 -> 130.9 mm
- net TX: track 0.00 -> 107.8 mm
- net RX: track 0.00 -> 104.6 mm
- net GND: track 0.00 -> 46.8 mm
- net SDA: track 0.00 -> 23.4 mm
- net SCL: track 0.00 -> 21.8 mm
- net 3.3V: track 0.00 -> 20.2 mm
- net 3V3OUT: track 0.00 -> 17.6 mm, vias 0 -> 2
- net X1: track 0.00 -> 11.8 mm
- net VBUS_SENSE: track 0.00 -> 11.7 mm
- net X0: track 0.00 -> 9.27 mm
- net N$3: track 0.00 -> 9.08 mm
- net N$4: track 0.00 -> 9.08 mm
- net USB_!RST: track 0.00 -> 8.86 mm
- net VIN: track 0.00 -> 8.70 mm
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- added copper zone on layer 1, net VIN

Commit message: Still routing!
Parts:
- removed R6: 10K, MF_Passives:R0603
- moved U14 333.3 mm to (335.8, 112.6), turned to 180 degrees
- moved U17 318.5 mm to (335.4, 44.5)
- moved R75 318.5 mm to (6.22, 51.9), turned to 0 degrees
- moved R69 318.4 mm to (6.22, 28.2), turned to 0 degrees
- moved R73 318.2 mm to (6.22, 44.1), turned to 0 degrees
- moved R70 318.2 mm to (6.22, 32.1), turned to 0 degrees
- moved R71 318.2 mm to (6.22, 36.2), turned to 0 degrees
- moved R74 318.0 mm to (6.22, 48.0), turned to 0 degrees
- moved R72 318.0 mm to (6.22, 40.1), turned to 0 degrees
- moved R76 316.9 mm to (6.22, 59.9), turned to 0 degrees
- moved U18 299.3 mm to (320.2, 30.9), turned to 0 degrees
- moved U16 295.2 mm to (320.9, 124.3), turned to 180 degrees
- moved R68 275.3 mm to (66.7, 6.73)
- moved R67 270.2 mm to (70.6, 6.60)
- moved R66 266.4 mm to (74.5, 6.60)
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Connections:
- net 3.3V: no longer R6.P$2
- net COIN_OUT: now also U14.2; no longer U14.6
- net DOOR_OUT: now also U14.5; no longer U14.3
- net ENTER_OUT: now also U14.3; no longer U14.5
- net PROP_!RST: no longer R6.P$1
- net R_FLIP_OUT: now also U14.7; no longer U14.1
- net SW_R_0: now also U15.7; no longer U15.15
- net SW_R_1: now also U15.6; no longer U15.1
- net SW_R_2: now also U15.5; no longer U15.2
- net SW_R_3: now also U15.4; no longer U15.3
- net SW_R_4: now also U15.3; no longer U15.4
- net SW_R_5: now also U15.2; no longer U15.5
- net SW_R_6: now also U15.1; no longer U15.6
- net SW_R_7: now also U15.15; no longer U15.7
- net TILT_OUT: now also U14.1; no longer U14.7
- net USER_0_OUT: now also U14.6; no longer U14.2
Routing:
- net DMD_11: track 0.00 -> 57.2 mm
- net DMD_9: track 0.00 -> 56.0 mm
- net DMD_7: track 0.00 -> 54.9 mm
- net DMD_5: track 0.00 -> 53.8 mm
- net ST_LI: track 0.00 -> 53.4 mm
- net DMD_3: track 0.00 -> 51.0 mm
- net SERVO_1: track 0.00 -> 48.7 mm
- net DMD_1: track 0.00 -> 46.6 mm
- net RGB_ROUT_L: track 0.00 -> 39.7 mm
- net SERVO_0: track 0.00 -> 39.6 mm
- net RGB_ROUT_R: track 0.00 -> 38.3 mm
- net RGB_BOUT_R: track 0.00 -> 38.2 mm
- net RGB_GOUT_R: track 0.00 -> 38.1 mm
- net DMD_13: track 0.00 -> 37.4 mm
- net PROP_AUX1: track 0.00 -> 36.9 mm
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- added copper zone on layer 1, net 12.0V_SW
- added copper zone on layer 1, net 3.3V
- added copper zone on layer 1, net 5.0V
- added copper zone on layer 1, net 5.0V_CUR
- added copper zone on layer 1, net 5.0V_SW
- added copper zone on layer 1, net GND
- added copper zone on layer 1, net VIN_CUR

Commit message: More work done. Fixed size issue.
Parts:
- moved R92 325.8 mm to (15.2, 87.4), turned to 180 degrees
- moved R91 324.2 mm to (15.2, 91.3), turned to 180 degrees
- moved R90 320.8 mm to (15.2, 95.2), turned to 180 degrees
- moved R89 319.3 mm to (15.2, 99.2), turned to 180 degrees
- moved R88 316.0 mm to (15.2, 103.1), turned to 180 degrees
- moved R87 314.6 mm to (15.2, 107.2), turned to 180 degrees
- moved R86 311.2 mm to (15.2, 111.1), turned to 180 degrees
- moved R85 310.1 mm to (15.2, 115.1), turned to 180 degrees
- moved R84 295.3 mm to (32.5, 91.4)
- moved R83 292.5 mm to (33.8, 94.5)
- moved R82 289.6 mm to (35.1, 91.4)
- moved R81 286.8 mm to (36.3, 94.5)
- moved R79 281.3 mm to (35.1, 111.5), turned to 270 degrees
- moved R80 281.3 mm to (36.3, 108.5), turned to 270 degrees
- moved R77 280.6 mm to (32.5, 111.5), turned to 270 degrees
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Routing:
- net GND: track 49.3 -> 156.7 mm, vias 0 -> 40
- net PROP_!RST: track 131.8 -> 48.1 mm
- net 3.3V: track 43.2 -> 106.6 mm
- net TX: track 107.8 -> 75.1 mm
- net RX: track 104.6 -> 72.8 mm
- net N$29: track 0.00 -> 30.1 mm
- net N$38: track 0.00 -> 29.5 mm
- net N$41: track 0.00 -> 29.3 mm
- net N$43: track 0.00 -> 28.8 mm
- net N$39: track 0.00 -> 26.6 mm
- net N$40: track 0.00 -> 26.4 mm
- net N$37: track 0.00 -> 26.2 mm
- net N$42: track 0.00 -> 26.0 mm
- net VIN: track 15.5 -> 11.9 mm
- net 5.0V: track 19.2 -> 15.8 mm
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Other:
- board size 359.2 x 152.3 mm -> 359.2 x 185.3 mm

Commit message: Almost done!
Parts:
- moved C23 77.8 mm to (78.6, 152.9), turned to 180 degrees
- moved U9 74.7 mm to (77.7, 150.1)
- moved U26 0.38 mm to (85.2, 111.4)
Connections:
- removed net P13: U1.14
- new net 3.3V_SENSE: 3.3V.P$1
- new net P7: U1.4
- net !RES!_PROP: now also U1.12; no longer U1.13
- net !RST!_PIC32: now also U1.9; no longer U1.10
- net 3.3V: no longer 3.3V.P$1
- net RX_PIC32: now also U1.11; no longer U1.4
- net RX_PROP: now also U1.14; no longer U1.11
- net TX_PIC32: now also U1.10; no longer U1.9
- net TX_PROP: now also U1.13; no longer U1.12
Routing:
- net 165_CLK: track 0.00 -> 611.3 mm, vias 0 -> 2
- net 165_LOAD: track 0.00 -> 598.9 mm, vias 0 -> 2
- net N$21: track 0.00 -> 379.0 mm, vias 0 -> 4
- net N$36: track 0.00 -> 302.8 mm
- net N$35: track 0.00 -> 302.6 mm
- net N$34: track 0.00 -> 302.4 mm
- net N$33: track 0.00 -> 302.2 mm
- net N$30: track 0.00 -> 302.1 mm
- net N$31: track 0.00 -> 302.0 mm
- net RX_PROP: track 0.00 -> 158.5 mm, vias 0 -> 1
- net TX_PROP: track 0.00 -> 155.8 mm, vias 0 -> 1
- net !RES!_PROP: track 0.00 -> 153.1 mm, vias 0 -> 1
- net RX_PIC32: track 0.00 -> 144.1 mm, vias 0 -> 1
- net TX_PIC32: track 0.00 -> 142.2 mm, vias 0 -> 1
- net !RST!_PIC32: track 0.00 -> 140.6 mm, vias 0 -> 1
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
Commit message: routing almost done.
Connections:
- removed net P16: U1.19
- removed net P17: U1.20
- removed net P18: U1.21
- removed net P19: U1.22
- removed net P20: U1.23
- removed net P21: U1.24
- new net P1: U1.42
- new net P2: U1.43
- new net P3: U1.44
- new net P4: U1.1
- new net P5: U1.2
- new net P6: U1.3
- net 165_CLK: now also U1.19; no longer U1.1
- net 165_DATA: now also U1.21; no longer U1.3
- net 165_LOAD: now also U1.20; no longer U1.2
- net 595_CLK: now also U1.22; no longer U1.42
- net 595_DATA: now also U1.24; no longer U1.44
- net 595_LAT: now also U1.23; no longer U1.43
Routing:
- net 595_LAT: track 0.00 -> 545.4 mm, vias 0 -> 4
- net 595_CLK: track 0.00 -> 532.4 mm, vias 0 -> 4
- net 165_LOAD: track 598.9 -> 883.2 mm, vias 2 -> 4
- net 165_CLK: track 611.3 -> 890.6 mm, vias 2 -> 4
- net 595_DATA: track 0.00 -> 238.4 mm, vias 0 -> 2
- net 165_DATA: track 0.00 -> 200.9 mm, vias 0 -> 2

Commit message: Almost done.
Need to change drill size.
Parts:
- added C26, C27, C28, C29, C30, C31, C32, C33, C34, C35, C36, C37, C38, C39: 0.1uF, MF_Passives:C0603
- !RES!_PROP, !RST!_PIC32, 12V, 3.3V, 50V, 5V, BACK_OUT, COIN_OUT, DMD_1, DMD_11, DMD_13, DMD_3, DMD_5, DMD_7, DMD_9, DOOR_OUT, ENTER_OUT, EXT_RGB_CLK, EXT_RGB_DATA, GI_R_0, GI_R_1, GI_R_10, GI_R_11, GI_R_12, GI_R_13, GI_R_14, GI_R_15, GI_R_2, GI_R_3, GI_R_4, GI_R_5, GI_R_6, GI_R_7, GI_R_8, GI_R_9, GND, LIGHT_C_0, LIGHT_C_1, LIGHT_C_2, LIGHT_C_3, LIGHT_C_4, LIGHT_C_5, LIGHT_C_6, LIGHT_C_7, LIGHT_R_0, LIGHT_R_1, LIGHT_R_2, LIGHT_R_3, LIGHT_R_4, LIGHT_R_5, LIGHT_R_6, LIGHT_R_7, L_FLIP_OUT, OPTO_1_, OPTO_2_, OPTO_3_, OPTO_4_, OPTO_5_, OPTO_6_, OPTO_7_, PROP_AUX0, PROP_AUX1, RGB_BOUT_L, RGB_BOUT_R, RGB_GOUT_L, RGB_GOUT_R, RGB_ROUT_L, RGB_ROUT_R, RX_PIC32, RX_PROP, R_FLIP_OUT, SD_CS, SD_DI, SD_DO, SD_SCLK, SERVO_0_, SERVO_1_, SERVO_2_, SERVO_3_, SERVO_4_, SOL_GND, SOL_PWR_0, SOL_PWR_1, SOL_PWR_10, SOL_PWR_11, SOL_PWR_12, SOL_PWR_13, SOL_PWR_14, SOL_PWR_15, SOL_PWR_16, SOL_PWR_17, SOL_PWR_18, SOL_PWR_19, SOL_PWR_2, SOL_PWR_20, SOL_PWR_21, SOL_PWR_22, SOL_PWR_23, SOL_PWR_3, SOL_PWR_4, SOL_PWR_5, SOL_PWR_6, SOL_PWR_7, SOL_PWR_8, SOL_PWR_9, ST_BU_OUT, ST_LI_, SW_C_0, SW_C_1, SW_C_2, SW_C_3, SW_C_4, SW_C_5, SW_C_6, SW_C_7, SW_R_0, SW_R_1, SW_R_2, SW_R_3, SW_R_4, SW_R_5, SW_R_6, SW_R_7, S_L, S_R, TILT_OUT, TX_PIC32, TX_PROP, USER_0_OUT: value (none) -> 0914-3-15-20-77-14-11-0
- moved C1 166.3 mm to (329.7, 109.2)
- moved C24 158.0 mm to (21.6, 24.8), turned to 270 degrees
- moved J2 4.70 mm to (9.53, 180.8), turned to 270 degrees
- moved TVS1 4.16 mm to (21.8, 177.9), turned to 90 degrees
- moved PICKIT3_IN 0.51 mm to (174.9, 183.4)
Connections:
- net 3.3V: now also C26.P$1, C27.P$1, C28.P$1, C29.P$1, C30.P$1, C31.P$1, C32.P$1, C33.P$1, C34.P$1, C35.P$1, C36.P$1, C37.P$1, C38.P$1, C39.P$1
- net 3.3V_SENSE: now also U9.P$3
- net GND: now also C26.P$2, C27.P$2, C28.P$2, C29.P$2, C30.P$2, C31.P$2, C32.P$2, C33.P$2, C34.P$2, C35.P$2, C36.P$2, C37.P$2, C38.P$2, C39.P$2
Routing:
- net 3.3V_SENSE: track 0.00 -> 55.5 mm
- net GND: track 276.0 -> 302.8 mm, vias 81 -> 89
- net 3.3V: track 98.0 -> 123.9 mm
- net VIN: track 16.0 -> 7.33 mm
- net N$33: track 302.2 -> 302.7 mm
- net N$31: track 302.0 -> 302.5 mm
- net N$30: track 302.1 -> 302.6 mm
- net N$36: track 302.8 -> 303.3 mm
- net N$35: track 302.6 -> 303.1 mm
- net N$34: track 302.4 -> 302.9 mm
