File: Hardware/Pinheck Test Jig/PinHeck Test Jig.brd (EAGLE design)
At the start: 359.2 x 185.3 mm, 327 parts, among them U1 P8X32A-Q44, U10 BSO080P03NS3E G, U11 BSO080P03NS3E G, U12 MF-DSC-SOT233-MMBT3904, U13 MF-DSC-SOT233-MMBT3904, U14 CD74HC595M96, U15 CD74HC595M96, U16 CD74HC165M96, U17 CD74HC165M96, U18 CD74HC165M96, U19 CD74HC165M96, U2 CAT24C512WI-GT3, U20 CD74HC165M96, U21 CD74HC165M96, U22 CD74HC165M96, U23 CD74HC165M96, U24 CD74HC165M96, U26 CD74HC165M96, U27 CD74HC165M96, U28 CD74HC165M96, U29 CD74HC165M96, U3 FT230XS, U30 CD74HC165M96, U4 IP4234CZ6, U5 NCP1117DT33G, U6 NCP1117DT50G, U7 INA139NA/3K, U8 INA139NA/3K, U9 MAX11613EUA+, X1 ABMM-6.000MHZ-B2-T

Commit message: Test Jig done.
Parts:
- added H18, H19, H20, H21: 2263-2, PP_Connectors:MOUNT_HOLE_120MIL
- H1, H10, H11, H12, H13, H14, H15, H16, H17, H2, H3, H4, H5, H6, H7, H8, H9: value MOUNT_HOLE150MIL -> 2263-2; device PP_Connectors:MOUNT_HOLE_150MIL -> PP_Connectors:MOUNT_HOLE_120MIL
- moved C6 6.73 mm to (136.3, 175.0)
- moved R4 6.73 mm to (143.1, 171.8)
- moved R3 6.73 mm to (140.7, 171.8)
- moved U2 6.73 mm to (142.2, 176.3)
- moved J1 0.89 mm to (87.1, 182.5)
Connections:
- net SHIELD: no longer J1.S1, J1.S2, J1.S7, J1.S8
Routing:
- net SHIELD: track 15.5 -> 23.0 mm
- net SDA: track 99.0 -> 92.3 mm
- net SCL: track 94.4 -> 87.7 mm
- net 3.3V: track 123.9 -> 129.8 mm, vias 0 -> 2
- net GND: track 302.8 -> 304.0 mm
- net V_USB_0: track 12.2 -> 13.1 mm
- net D+_USB: track 3.23 -> 4.11 mm
- net D-_USB: track 3.22 -> 4.11 mm
