File: Hardware/Pinheck Test Jig/PinHeck Test Jig.sch (EAGLE design)
At the start: 194 parts, among them SW1 MF-SW-TACT-6MM, U1 P8X32A-Q44, U2 CAT24C512WI-GT3, U3 FT230XS, U4 IP4234CZ6, U5 NCP1117DT33G, U6 NCP1117DT50G, X1 ABMM-6.000MHZ-B2-T

Commit message: Added AUX, and RGB LED Board. Working on Test Jib.
Parts:
- removed R1, R2: 10K, MF_Passives:RESISTOR_0805
- removed SD1: (no value), PP_Connectors:SD_CARD_SD-RSMT-2-MQ
- added C21, C22, C23, C24: 0.1uF, PP_Passives:CAPACITOR_NON_POLAR_0805
- added R14, R15: RL73H2BR10FTD, PP_Passives:RESISTOR_1206
- added R16, R17: ERJ-6ENF3002V, PP_Passives:RESISTOR_0805
- added R18, R19, R20, R21: 10K, PP_Passives:RESISTOR_0805
- added TVS1: V18AUMLA2220H, PP_Passives:TVS_DIODE_2220
- added U10, U11: BSO080P03NS3E G, PP_DiscreteSemi:MOSFET_P-CHANNEL_SINGLE_P3-POWER
- added U12, U13: MF-DSC-SOT233-MMBT3904, PP_DiscreteSemi:BJT_NPN_SINGLE_SOT-23
- added U14, U15: CD74HC595M96, PP_DigitalIC:CD74HC595M96
- added U16, U17, U18, U19, U20, U21, U22, U23, U24, U25, U26, U27, U28, U29, U30, U31: CD74HC165M96, PP_DigitalIC:CD74HC165M96
- added U7, U8: INA139NA/3K, PP_AnalogIC:INA169SOT-23-5
- added U9: MAX11613EUA+, PP_AnalogIC:MAX11613EUA+
- C1: value 1uF -> 0.1uF; device MF_Passives:CAPACITOR_NP_0805 -> PP_Passives:CAPACITOR_NON_POLAR_0805
Connections:
- net IN_OPTO_0 renamed P27
- net IN_OPTO_1 renamed P26
- net IN_OPTO_2 renamed P25
- net IN_OPTO_3 renamed P24
- net IN_OPTO_4 renamed P23
- net IN_OPTO_5 renamed P22
- net IN_OPTO_6 renamed P21
- net IN_OPTO_7 renamed P20
- net LCD_RES renamed P19
- net OUT_OPTO_0 renamed P18
- net OUT_OPTO_1 renamed P17
- net OUT_OPTO_10 renamed P8
- net OUT_OPTO_11 renamed P7
- net OUT_OPTO_12 renamed P6
- net OUT_OPTO_13 renamed P5
- net OUT_OPTO_14 renamed P4
- net OUT_OPTO_15 renamed P3
- net OUT_OPTO_16 renamed P2
- net OUT_OPTO_17 renamed P1
- net OUT_OPTO_2 renamed P16
- net OUT_OPTO_3 renamed P15
- net OUT_OPTO_4 renamed P14
- net OUT_OPTO_5 renamed P13
- net OUT_OPTO_6 renamed P12
- net OUT_OPTO_7 renamed P11
- net OUT_OPTO_8 renamed P10
- net OUT_OPTO_9 renamed P9
- removed net 12V_IN: 12V.P$1
- removed net 5V_IN: 5V.P$1
- new net 12.0V_SW: 12V.P$1, U10.SOURCE
- new net 165_CLK: U16.CLK, U17.CLK, U18.CLK, U19.CLK, U20.CLK, U21.CLK, U22.CLK, U23.CLK, U24.CLK, U25.CLK, U26.CLK, U27.CLK, U28.CLK, U29.CLK, U30.CLK, U31.CLK
- new net 165_DATA: U16.QH
- new net 165_LOAD: U16.LAT, U17.LAT, U18.LAT, U19.LAT, U20.LAT, U21.LAT, U22.LAT, U23.LAT, U24.LAT, U25.LAT, U26.LAT, U27.LAT, U28.LAT, U29.LAT, U30.LAT, U31.LAT
- new net 5.0V_CUR: R15.2, R20.1, U11.DRAIN, U8.VIN-
- new net 5.0V_SW: 5V.P$1, U11.SOURCE
- new net 595_CLK: U14.SHCP, U15.SHCP
- new net 595_DATA: U14.DS
- new net 595_LAT: U14.STCP, U15.STCP
- new net A_0: C21.1, R16.2, U7.OUT, U9.A_0
- new net A_1: C22.1, R17.2, U8.OUT, U9.A_1
- new net N$11: R18.2, U10.GATE, U12.COLLECTOR
- new net N$12: R20.2, U11.GATE, U13.COLLECTOR
- new net N$13: R19.2, U12.BASE
- new net N$14: U20.SER, U21.QH
- new net N$15: R21.2, U13.BASE
- new net N$16: U21.SER, U22.QH
- new net N$17: U22.SER, U23.QH
- new net N$18: U23.SER, U24.QH
- new net N$19: U24.SER, U25.QH
- new net N$20: U16.D7
- new net N$21: U14.Q7S, U15.DS
- new net N$22: U16.SER, U17.QH
- new net N$23: U25.SER, U26.QH
- new net N$24: U17.SER, U18.QH
- new net N$25: U26.SER, U27.QH
- new net N$26: U27.SER, U28.QH
- new net N$27: U28.SER, U29.QH
- new net N$28: U29.SER, U30.QH
- new net N$29: U30.SER, U31.QH
- new net PWR_ON: R19.1, R21.1, U1.P0
- new net VIN_CUR: R14.2, R18.1, U10.DRAIN, U7.VIN-
- net 3.3V: now also C1.1, C23.1, C24.1, U14.MR, U14.VCC, U15.MR, U15.VCC, U16.VCC, U17.VCC, U18.VCC, U19.VCC, U20.VCC, U21.VCC, U22.VCC, U23.VCC, U24.VCC, U25.VCC, U26.VCC, U27.VCC, U28.VCC, U29.VCC, U30.VCC, U31.VCC, U7.V+, U8.V+, U9.VCC; no longer C1.P$2, R1.P$1, R2.P$1, SD1.3.3V
- net 5.0V: now also R15.1, U8.VIN+
- net BACK_OUT: now also U14.Q4
- net COIN_OUT: now also U14.Q6
- net DMD_1: now also U29.D2
- net DMD_11: now also U29.D7
- net DMD_13: now also U30.D0
- net DMD_3: now also U29.D3
- net DMD_5: now also U29.D4
- net DMD_7: now also U29.D5
- net DMD_9: now also U29.D6
- net DOOR_OUT: now also U14.Q3
- net ENTER_OUT: now also U14.Q5
- net EXT_RGB_CLK: now also U28.D0
- net EXT_RGB_DATA: now also U28.D1
- net GI15: now also U18.D0
- net GI_R_0: now also U17.D7
- net GI_R_1: now also U17.D6
- net GI_R_10: now also U18.D5
- net GI_R_11: now also U18.D4
- net GI_R_12: now also U18.D3
- net GI_R_13: now also U18.D2
- net GI_R_14: now also U18.D1
- net GI_R_2: now also U17.D5
- net GI_R_3: now also U17.D4
- net GI_R_4: now also U17.D3
- net GI_R_5: now also U17.D2
- net GI_R_6: now also U17.D1
- net GI_R_7: now also U17.D0
- net GI_R_8: now also U18.D7
- net GI_R_9: now also U18.D6
- net GND: now also C1.2, C21.2, C22.2, C23.2, C24.2, R16.1, R17.1, TVS1.P$2, U12.EMITTER, U13.EMITTER, U14.GND, U14.OE, U15.GND, U15.OE, U16.C_INH, U16.GND, U17.C_INH, U17.GND, U18.C_INH, U18.GND, U19.C_INH, U19.GND, U20.C_INH, U20.GND, U21.C_INH, U21.GND, U22.C_INH, U22.GND, U23.C_INH, U23.GND, U24.C_INH, U24.GND, U25.C_INH, U25.GND, U26.C_INH, U26.GND, U27.C_INH, U27.GND, U28.C_INH, U28.GND, U29.C_INH, U29.GND, U30.C_INH, U30.GND, U31.C_INH, U31.GND, U7.GND, U8.GND, U9.GND; no longer C1.P$1, SD1.GND
- net LIGHT_C_0: now also U24.D7, U25.D7
- net LIGHT_C_1: now also U24.D6, U25.D6
- net LIGHT_C_2: now also U24.D5, U25.D5
- net LIGHT_C_3: now also U24.D4, U25.D4
- net LIGHT_C_4: now also U24.D3, U25.D3
- net LIGHT_C_5: now also U24.D2, U25.D2
- net LIGHT_C_6: now also U24.D1, U25.D1
- net LIGHT_C_7: now also U24.D0, U25.D0
- net LIGHT_R_0: now also U23.D7
- net LIGHT_R_1: now also U23.D6
- net LIGHT_R_2: now also U23.D5
- net LIGHT_R_3: now also U23.D4
- net LIGHT_R_4: now also U23.D3
- net LIGHT_R_5: now also U23.D2
- net LIGHT_R_6: now also U23.D1
- net LIGHT_R_7: now also U23.D0
- net L_FLIP_OUT: now also U14.Q0
- net N$1: now also U18.SER, U19.QH; no longer R1.P$2, SD1.RW
- net N$2: now also U19.SER, U20.QH; no longer R2.P$2, SD1.IRQ
- net OPTO_1: now also U26.D0
- net OPTO_2: now also U26.D1
- net OPTO_3: now also U26.D2
- net OPTO_4: now also U26.D3
- net OPTO_5: now also U26.D4
- net OPTO_6: now also U26.D5
- net OPTO_7: now also U26.D6
- net PROP_AUX0: now also U28.D2
- net PROP_AUX1: now also U28.D3
- net RGB_BOUT_L: now also U29.D1
- net RGB_BOUT_R: now also U28.D6
- net RGB_GOUT_L: now also U29.D0
- net RGB_GOUT_R: now also U28.D5
- net RGB_ROUT_L: now also U28.D7
- net RGB_ROUT_R: now also U28.D4
- net R_FLIP_OUT: now also U14.Q1
- net SCL: now also U9.SCL
- net SDA: now also U9.SDA
- net SD_CS: now also U16.D0; no longer SD1.CS
- net SD_DI: now also U16.D1; no longer SD1.DI
- net SD_DO: now also U16.D3; no longer SD1.D0
- net SD_SCLK: now also U16.D2; no longer SD1.SCLK
- net SERVO_0: now also U27.D0
- net SERVO_1: now also U27.D1
- net SERVO_2: now also U27.D2
- net SERVO_3: now also U27.D3
- net SERVO_4: now also U27.D4
- net SOL_PWR_0: now also U21.D7
- net SOL_PWR_1: now also U21.D6
- net SOL_PWR_10: now also U20.D5
- net SOL_PWR_11: now also U20.D4
- net SOL_PWR_12: now also U20.D3
- net SOL_PWR_13: now also U20.D2
- net SOL_PWR_14: now also U20.D1
- net SOL_PWR_15: now also U20.D0
- net SOL_PWR_16: now also U19.D7
- net SOL_PWR_17: now also U19.D6
- net SOL_PWR_18: now also U19.D5
- net SOL_PWR_19: now also U19.D4
- net SOL_PWR_2: now also U21.D5
- net SOL_PWR_20: now also U19.D3
- net SOL_PWR_21: now also U19.D2
- net SOL_PWR_22: now also U19.D1
- net SOL_PWR_23: now also U19.D0
- net SOL_PWR_3: now also U21.D4
- net SOL_PWR_4: now also U21.D3
- net SOL_PWR_5: now also U21.D2
- net SOL_PWR_6: now also U21.D1
- net SOL_PWR_7: now also U21.D0
- net SOL_PWR_8: now also U20.D7
- net SOL_PWR_9: now also U20.D6
- net ST_LI: now also U16.D6
- net SW_C_0: now also U22.D0, U31.D0
- net SW_C_1: now also U22.D1, U30.D1, U31.D1
- net SW_C_2: now also U22.D2, U30.D2, U31.D2
- net SW_C_3: now also U22.D3, U30.D3, U31.D3
- net SW_C_4: now also U22.D4, U30.D4, U31.D4
- net SW_C_5: now also U22.D5, U30.D5, U31.D5
- net SW_C_6: now also U22.D6, U30.D6, U31.D6
- net SW_C_7: now also U22.D7, U30.D7, U31.D7
- net SW_R_0: now also U15.Q0
- net SW_R_1: now also U15.Q1
- net SW_R_2: now also U15.Q2
- net SW_R_3: now also U15.Q3
- net SW_R_4: now also U15.Q4
- net SW_R_5: now also U15.Q5
- net SW_R_6: now also U15.Q6
- net SW_R_7: now also U15.Q7
- net S_L: now also U16.D4
- net S_R: now also U16.D5
- net TILT_OUT: now also U14.Q7
- net USB_!RST: no longer U1.P0
- net USER_0_OUT: now also U14.Q2
- net VIN: now also R14.1, TVS1.P$1, U7.VIN+
Other:
- moved on the sheet: C1, C13, C14, C15, C16, C17, C18, C19, C20, J2, U5, U6

Commit message: Jig Schematic Done.
Parts:
- removed PIC32_UART, PICKIT3, PROP_UART: (no value), PP_Connectors:CON_01X06_2.54MM_PIN_HEADER
- removed U25, U31: CD74HC165M96, PP_DigitalIC:CD74HC165M96
- added !MCLR!/VPP, !RES!_PROP, !RST!_PIC32, ICSPCLK, ICSPDAT, PGM, RX_PIC32, RX_PROP, TX_PIC32, TX_PROP, VDD, VSS: (no value), PP_Connectors:POGO_PIN_0914-3-15-20-77-14-11-0
- added R1, R100, R2, R22, R23, R24, R25, R26, R27, R28, R29, R31, R32, R33, R34, R35, R36, R37, R38, R39, R40, R41, R42, R43, R44, R45, R46, R47, R48, R49, R50, R51, R52, R53, R54, R55, R56, R57, R58, R59, R60, R61, R62, R63, R64, R65, R66, R67, R68, R69, R70, R71, R72, R73, R74, R75, R76, R77, R78, R79, R80, R81, R82, R83, R84, R93, R94, R97, R98, R99: 10K, MF_Passives:RESISTOR_0603
- added R85, R86, R87, R88, R89, R90, R91, R92: 30K, MF_Passives:RESISTOR_0603
- PICKIT3_IN: LABEL01 (none) -> !MCLR!/VPP; LABEL02 (none) -> VDD; LABEL03 (none) -> VSS; LABEL04 (none) -> ICSPDAT; LABEL05 (none) -> ICSPCLK; LABEL06 (none) -> PGM
Connections:
- removed net N$19: U24.SER, U25.QH
- removed net N$20: U16.D7
- removed net P1: U1.P1
- removed net P10: U1.P10
- removed net P11: U1.P11
- removed net P12: U1.P12
- removed net P2: U1.P2
- removed net P3: U1.P3
- removed net P4: U1.P4
- removed net P5: U1.P5
- removed net P6: U1.P6
- removed net P7: U1.P7
- removed net P8: U1.P8
- removed net P9: U1.P9
- removed net SOL_GND: SOL_GND.P$1
- new net !RES!_PROP: !RES!_PROP.P$1, U1.P12
- new net !RST!_PIC32: !RST!_PIC32.P$1, U1.P9
- new net N$30: !MCLR!/VPP.P$1, PICKIT3_IN.1
- new net N$31: PICKIT3_IN.2, VDD.P$1
- new net N$33: PICKIT3_IN.3, VSS.P$1
- new net N$34: ICSPDAT.P$1, PICKIT3_IN.4
- new net N$35: ICSPCLK.P$1, PICKIT3_IN.5
- new net N$36: PGM.P$1, PICKIT3_IN.6
- new net N$37: R83.P$2, R91.P$1, U24.D1
- new net N$38: R82.P$2, R90.P$1, U24.D2
- new net N$39: R81.P$2, R89.P$1, U24.D3
- new net N$40: R80.P$2, R88.P$1, U24.D4
- new net N$41: R79.P$2, R87.P$1, U24.D5
- new net N$42: R78.P$2, R86.P$1, U24.D6
- new net N$43: R77.P$2, R85.P$1, U24.D7
- new net RX_PIC32: RX_PIC32.P$1, U1.P7
- new net RX_PROP: RX_PROP.P$1, U1.P10
- new net TX_PIC32: TX_PIC32.P$1, U1.P8
- new net TX_PROP: TX_PROP.P$1, U1.P11
- net 165_CLK: now also U1.P4; no longer U25.CLK, U31.CLK
- net 165_DATA: now also U1.P6
- net 165_LOAD: now also U1.P5; no longer U25.LAT, U31.LAT
- net 3.3V: now also R1.P$1, R100.P$1, R2.P$1, R22.P$1, R23.P$1, R24.P$1, R25.P$1, R26.P$1, R27.P$1, R28.P$1, R29.P$1, R31.P$1, R32.P$1, R33.P$1, R34.P$1, R35.P$1, R36.P$1, R37.P$1, R38.P$1, R39.P$1, R40.P$1, R41.P$1, R42.P$1, R43.P$1, R44.P$1, R45.P$1, R46.P$1, R47.P$1, R48.P$1, R49.P$1, R50.P$1, R51.P$1, R52.P$1, R53.P$1, R54.P$1, R55.P$1, R56.P$1, R57.P$1, R58.P$1, R59.P$1, R60.P$1, R61.P$1, R62.P$1, R63.P$1, R64.P$1, R65.P$1, R66.P$1, R67.P$1, R68.P$1, R69.P$1, R70.P$1, R71.P$1, R72.P$1, R73.P$1, R74.P$1, R75.P$1, R76.P$1, R93.P$1, R94.P$1, R97.P$1, R98.P$1, R99.P$1; no longer U25.VCC, U31.VCC
- net 595_CLK: now also U1.P1
- net 595_DATA: now also U1.P3
- net 595_LAT: now also U1.P2
- net GI15: now also R28.P$2
- net GI_R_0: now also R27.P$2
- net GI_R_1: now also R26.P$2
- net GI_R_10: now also R34.P$2
- net GI_R_11: now also R33.P$2
- net GI_R_12: now also R32.P$2
- net GI_R_13: now also R31.P$2
- net GI_R_14: now also R29.P$2
- net GI_R_2: now also R25.P$2
- net GI_R_3: now also R24.P$2
- net GI_R_4: now also R23.P$2
- net GI_R_5: now also R22.P$2
- net GI_R_6: now also R2.P$2
- net GI_R_7: now also R1.P$2
- net GI_R_8: now also R36.P$2
- net GI_R_9: now also R35.P$2
- net GND: now also R77.P$1, R78.P$1, R79.P$1, R80.P$1, R81.P$1, R82.P$1, R83.P$1, R84.P$1, SOL_GND.P$1; no longer U25.C_INH, U25.GND, U31.C_INH, U31.GND
- net LIGHT_C_0: now also R85.P$2; no longer U24.D7, U25.D7
- net LIGHT_C_1: now also R86.P$2; no longer U24.D6, U25.D6
- net LIGHT_C_2: now also R87.P$2; no longer U24.D5, U25.D5
- net LIGHT_C_3: now also R88.P$2; no longer U24.D4, U25.D4
- net LIGHT_C_4: now also R89.P$2; no longer U24.D3, U25.D3
- net LIGHT_C_5: now also R90.P$2; no longer U24.D2, U25.D2
- net LIGHT_C_6: now also R91.P$2; no longer U24.D1, U25.D1
- net LIGHT_C_7: now also R92.P$2; no longer U24.D0, U25.D0
- net LIGHT_R_0: now also R76.P$2
- net LIGHT_R_1: now also R75.P$2
- net LIGHT_R_2: now also R74.P$2
- net LIGHT_R_3: now also R73.P$2
- net LIGHT_R_4: now also R72.P$2
- net LIGHT_R_5: now also R71.P$2
- net LIGHT_R_6: now also R70.P$2
- net LIGHT_R_7: now also R69.P$2
- net N$23: now also U24.SER; no longer U25.SER
- net N$29: now also R84.P$2, R92.P$1, U24.D0; no longer U30.SER, U31.QH
- net RGB_BOUT_L: now also R94.P$2
- net RGB_BOUT_R: now also R99.P$2
- net RGB_GOUT_L: now also R93.P$2
- net RGB_GOUT_R: now also R98.P$2
- net RGB_ROUT_L: now also R100.P$2
- net RGB_ROUT_R: now also R97.P$2
- net SOL_PWR_0: now also R60.P$2
- net SOL_PWR_1: now also R59.P$2
- net SOL_PWR_10: now also R50.P$2
- net SOL_PWR_11: now also R49.P$2
- net SOL_PWR_12: now also R48.P$2
- net SOL_PWR_13: now also R47.P$2
- net SOL_PWR_14: now also R46.P$2
- net SOL_PWR_15: now also R45.P$2
- net SOL_PWR_16: now also R44.P$2
- net SOL_PWR_17: now also R43.P$2
- net SOL_PWR_18: now also R42.P$2
- net SOL_PWR_19: now also R41.P$2
- net SOL_PWR_2: now also R58.P$2
- net SOL_PWR_20: now also R40.P$2
- net SOL_PWR_21: now also R39.P$2
- net SOL_PWR_22: now also R38.P$2
- net SOL_PWR_23: now also R37.P$2
- net SOL_PWR_3: now also R57.P$2
- net SOL_PWR_4: now also R56.P$2
- net SOL_PWR_5: now also R55.P$2
- net SOL_PWR_6: now also R54.P$2
- net SOL_PWR_7: now also R53.P$2
- net SOL_PWR_8: now also R52.P$2
- net SOL_PWR_9: now also R51.P$2
- net SW_C_0: now also R61.P$2; no longer U31.D0
- net SW_C_1: now also R62.P$2; no longer U30.D1, U31.D1
- net SW_C_2: now also R63.P$2; no longer U30.D2, U31.D2
- net SW_C_3: now also R64.P$2; no longer U30.D3, U31.D3
- net SW_C_4: now also R65.P$2; no longer U30.D4, U31.D4
- net SW_C_5: now also R66.P$2; no longer U30.D5, U31.D5
- net SW_C_6: now also R67.P$2; no longer U30.D6, U31.D6
- net SW_C_7: now also R68.P$2; no longer U30.D7, U31.D7
Other:
- moved on the sheet: PICKIT3_IN, U17, U18, U19, U20, U21, U22, U23, U24, U26, U27, U28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

Commit message: Routing Test Jig.
Parts:
- removed SW1: MF-SW-TACT-6MM, MF_Switches:TACT_6MM
- added C25: 0.1uF, MF_Passives:CAPACITOR_NP_0603
Connections:
- removed net N$7: C9.P$2, R6.P$1, SW1.P$3
- net 3.3V: now also C25.P$1
- net GND: now also C25.P$2
- net PROP_!RST: now also C9.P$2, R6.P$1; no longer SW1.P$2
Other:
- moved on the sheet: C9
Changed lines of the file:
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@@
 <part name="U1" library="MF_IC_Digital" deviceset="P8X32A" device="-Q44"/>
 <part name="X1" library="MF_Frequency_Control" deviceset="XTL" device="_7MMX5MM" value="ABMM-6.000MHZ-B2-T"/>
-<part name="SW1" library="MF_Switches" deviceset="TACT" device="_6MM" value="MF-SW-TACT-6MM"/>
 <part name="C2" library="MF_Passives" deviceset="CAPACITOR_NP" device="_0603" value="0.1uF"/>
 <part name="C3" library="MF_Passives" deviceset="CAPACITOR_NP" device="_0603" value="0.1uF"/>
@@
 <part name="R93" library="MF_Passives" deviceset="RESISTOR" device="_0603" value="10K"/>
 <part name="R94" library="MF_Passives" deviceset="RESISTOR" device="_0603" value="10K"/>
+<part name="C25" library="MF_Passives" deviceset="CAPACITOR_NP" device="_0603" value="0.1uF"/>
 </parts>
 <sheets>
@@
 <instance part="U1" gate="G$1" x="101.6" y="167.64"/>
 <instance part="X1" gate="G$1" x="132.08" y="170.18" rot="MR180"/>
-<instance part="SW1" gate="G$1" x="68.58" y="162.56"/>
 <instance part="C2" gate="G$1" x="93.98" y="101.6"/>
 <instance part="C3" gate="G$1" x="104.14" y="101.6"/>
@@
 <instance part="J1" gate="G$1" x="-129.54" y="160.02"/>
 <instance part="L1" gate="G$1" x="-111.76" y="132.08"/>
-<instance part="C9" gate="G$1" x="45.72" y="160.02" rot="R90"/>
+<instance part="C9" gate="G$1" x="45.72" y="165.1" rot="R90"/>
 <instance part="C10" gate="G$1" x="-30.48" y="144.78"/>
 <instance part="C11" gate="G$1" x="-45.72" y="144.78"/>
@@
 <instance part="R93" gate="G$1" x="198.12" y="-358.14" rot="R270"/>
 <instance part="R94" gate="G$1" x="203.2" y="-358.14" rot="R270"/>
+<instance part="C25" gate="G$1" x="134.62" y="101.6"/>
 </instances>
 <busses>
@@
 <segment>
 <pinref part="U1" gate="G$1" pin="VSS"/>
-<wire x1="119.38" y1="114.3" x2="132.08" y2="114.3" width="0.1524" layer="91"/>
+<wire x1="119.38" y1="114.3" x2="142.24" y2="114.3" width="0.1524" layer="91"/>
 <label x="121.92" y="114.3" size="1.016" layer="95" font="vector"/>
 <pinref part="C2" gate="G$1" pin="P$2"/>
@@
 <wire x1="104.14" y1="93.98" x2="114.3" y2="93.98" width="0.1524" layer="91"/>
 <wire x1="114.3" y1="93.98" x2="124.46" y2="93.98" width="0.1524" layer="91"/>
-<wire x1="124.46" y1="93.98" x2="132.08" y2="93.98" width="0.1524" layer="91"/>
-<wire x1="132.08" y1="93.98" x2="132.08" y2="114.3" width="0.1524" layer="91"/>
+<wire x1="124.46" y1="93.98" x2="134.62" y2="93.98" width="0.1524" layer="91"/>
+<wire x1="134.62" y1="93.98" x2="142.24" y2="93.98" width="0.1524" layer="91"/>
+<wire x1="142.24" y1="93.98" x2="142.24" y2="114.3" width="0.1524" layer="91"/>
 <pinref part="C5" gate="G$1" pin="P$2"/>
 <wire x1="124.46" y1="96.52" x2="124.46" y2="93.98" width="0.1524" layer="91"/>
@@
 <wire x1="93.98" y1="93.98" x2="93.98" y2="91.44" width="0.1524" layer="91"/>
 <junction x="93.98" y="93.98"/>
+<pinref part="C25" gate="G$1" pin="P$2"/>
+<wire x1="134.62" y1="93.98" x2="134.62" y2="96.52" width="0.1524" layer="91"/>
 </segment>
 <segment>
@@
 <wire x1="83.82" y1="114.3" x2="83.82" y2="182.88" width="0.1524" layer="91"/>
 <wire x1="83.82" y1="182.88" x2="81.28" y2="182.88" width="0.1524" layer="91"/>
+<pinref part="C25" gate="G$1" pin="P$1"/>
+<wire x1="124.46" y1="109.22" x2="134.62" y2="109.22" width="0.1524" layer="91"/>
+<wire x1="134.62" y1="109.22" x2="134.62" y2="106.68" width="0.1524" layer="91"/>
+<junction x="124.46" y="109.22"/>
 </segment>
 <segment>
@@
 <segment>
 <pinref part="U1" gate="G$1" pin="RES'"/>
-<pinref part="SW1" gate="G$1" pin="P$2"/>
 <wire x1="99.06" y1="165.1" x2="81.28" y2="165.1" width="0.1524" layer="91"/>
 <label x="86.36" y="165.1" size="1.016" layer="95" font="vector"/>
 <pinref part="R5" gate="G$1" pin="P$1"/>
-<wire x1="81.28" y1="165.1" x2="71.12" y2="165.1" width="0.1524" layer="91"/>
 <wire x1="81.28" y1="170.18" x2="81.28" y2="165.1" width="0.1524" layer="91"/>
 <junction x="81.28" y="165.1"/>
+<pinref part="C9" gate="G$1" pin="P$2"/>
+<wire x1="50.8" y1="165.1" x2="55.88" y2="165.1" width="0.1524" layer="91"/>
+<pinref part="R6" gate="G$1" pin="P$1"/>
+<wire x1="55.88" y1="165.1" x2="81.28" y2="165.1" width="0.1524" layer="91"/>
+<wire x1="55.88" y1="170.18" x2="55.88" y2="165.1" width="0.1524" layer="91"/>
+<junction x="55.88" y="165.1"/>
 </segment>
 </net>
@@
 <segment>
 <pinref part="C9" gate="G$1" pin="P$1"/>
-<wire x1="30.48" y1="160.02" x2="40.64" y2="160.02" width="0.1524" layer="91"/>
-<label x="30.48" y="160.02" size="1.016" layer="95" font="vector"/>
-</segment>
-</net>
-<net name="N$7" class="0">
-<segment>
-<pinref part="C9" gate="G$1" pin="P$2"/>
-<pinref part="SW1" gate="G$1" pin="P$3"/>
-<wire x1="50.8" y1="160.02" x2="55.88" y2="160.02" width="0.1524" layer="91"/>
-<pinref part="R6" gate="G$1" pin="P$1"/>
-<wire x1="55.88" y1="160.02" x2="66.04" y2="160.02" width="0.1524" layer="91"/>
-<wire x1="55.88" y1="170.18" x2="55.88" y2="160.02" width="0.1524" layer="91"/>
-<junction x="55.88" y="160.02"/>
+<wire x1="30.48" y1="165.1" x2="40.64" y2="165.1" width="0.1524" layer="91"/>
+<label x="30.48" y="165.1" size="1.016" layer="95" font="vector"/>
 </segment>
 </net>
