File: Hardware/Pinheck Test Jig/PinHeck Test Jig.sch (EAGLE design)
At the start: 314 parts, among them U1 P8X32A-Q44, U10 BSO080P03NS3E G, U11 BSO080P03NS3E G, U12 MF-DSC-SOT233-MMBT3904, U13 MF-DSC-SOT233-MMBT3904, U14 CD74HC595M96, U15 CD74HC595M96, U16 CD74HC165M96, U17 CD74HC165M96, U18 CD74HC165M96, U19 CD74HC165M96, U2 CAT24C512WI-GT3, U20 CD74HC165M96, U21 CD74HC165M96, U22 CD74HC165M96, U23 CD74HC165M96, U24 CD74HC165M96, U26 CD74HC165M96, U27 CD74HC165M96, U28 CD74HC165M96, U29 CD74HC165M96, U3 FT230XS, U30 CD74HC165M96, U4 IP4234CZ6, U5 NCP1117DT33G, U6 NCP1117DT50G, U7 INA139NA/3K, U8 INA139NA/3K, U9 MAX11613EUA+, X1 ABMM-6.000MHZ-B2-T

Commit message: Still routing!
Parts:
- removed R6: 10K, MF_Passives:RESISTOR_0603
Connections:
- net 3.3V: no longer R6.P$2
- net COIN_OUT: now also U14.Q2; no longer U14.Q6
- net DOOR_OUT: now also U14.Q5; no longer U14.Q3
- net ENTER_OUT: now also U14.Q3; no longer U14.Q5
- net PROP_!RST: no longer R6.P$1
- net R_FLIP_OUT: now also U14.Q7; no longer U14.Q1
- net SW_R_0: now also U15.Q7; no longer U15.Q0
- net SW_R_1: now also U15.Q6; no longer U15.Q1
- net SW_R_2: now also U15.Q5; no longer U15.Q2
- net SW_R_3: now also U15.Q4; no longer U15.Q3
- net SW_R_4: now also U15.Q3; no longer U15.Q4
- net SW_R_5: now also U15.Q2; no longer U15.Q5
- net SW_R_6: now also U15.Q1; no longer U15.Q6
- net SW_R_7: now also U15.Q0; no longer U15.Q7
- net TILT_OUT: now also U14.Q1; no longer U14.Q7
- net USER_0_OUT: now also U14.Q6; no longer U14.Q2
Other:
- moved on the sheet: C9
Changed lines of the file:
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@@
 <?xml version="1.0" encoding="utf-8"?>
 <!DOCTYPE eagle SYSTEM "eagle.dtd">
-<eagle version="6.6.0">
+<eagle version="6.5.0">
 <drawing>
 <settings>
@@
 <part name="C6" library="MF_Passives" deviceset="CAPACITOR_NP" device="_0603" value="0.1uF"/>
 <part name="R5" library="MF_Passives" deviceset="RESISTOR" device="_0603" value="10K"/>
-<part name="R6" library="MF_Passives" deviceset="RESISTOR" device="_0603" value="10K"/>
 <part name="U3" library="MF_IC_Digital" deviceset="FT230X" device="S"/>
 <part name="U4" library="PP_Passives" deviceset="IP4234CZ6" device="" value="IP4234CZ6"/>
@@
 <instance part="C6" gate="G$1" x="190.5" y="172.72"/>
 <instance part="R5" gate="G$1" x="81.28" y="175.26" rot="R90"/>
-<instance part="R6" gate="G$1" x="55.88" y="175.26" rot="R90"/>
 <instance part="U3" gate="G$1" x="-17.78" y="165.1"/>
 <instance part="U4" gate="G$1" x="-91.44" y="152.4" rot="R90"/>
@@
 <instance part="J1" gate="G$1" x="-129.54" y="160.02"/>
 <instance part="L1" gate="G$1" x="-111.76" y="132.08"/>
-<instance part="C9" gate="G$1" x="45.72" y="165.1" rot="R90"/>
+<instance part="C9" gate="G$1" x="68.58" y="165.1" rot="R90"/>
 <instance part="C10" gate="G$1" x="-30.48" y="144.78"/>
 <instance part="C11" gate="G$1" x="-45.72" y="144.78"/>
@@
 <pinref part="R5" gate="G$1" pin="P$2"/>
 <wire x1="81.28" y1="180.34" x2="81.28" y2="182.88" width="0.1524" layer="91"/>
-<wire x1="81.28" y1="182.88" x2="55.88" y2="182.88" width="0.1524" layer="91"/>
-<pinref part="R6" gate="G$1" pin="P$2"/>
-<wire x1="55.88" y1="182.88" x2="55.88" y2="180.34" width="0.1524" layer="91"/>
-<label x="58.42" y="182.88" size="1.016" layer="95" font="vector"/>
 <pinref part="U$12" gate="G$1" pin="P$1"/>
 <wire x1="81.28" y1="182.88" x2="81.28" y2="185.42" width="0.1524" layer="91"/>
@@
 </segment>
 <segment>
-<pinref part="U15" gate="G$1" pin="Q6"/>
-<wire x1="111.76" y1="12.7" x2="101.6" y2="12.7" width="0.1524" layer="91"/>
-<label x="106.68" y="12.7" size="1.016" layer="95" font="vector"/>
+<pinref part="U15" gate="G$1" pin="Q1"/>
+<wire x1="101.6" y1="25.4" x2="111.76" y2="25.4" width="0.1524" layer="91"/>
+<label x="106.68" y="25.4" size="1.016" layer="95" font="vector"/>
 </segment>
 </net>
@@
 </segment>
 <segment>
-<pinref part="U15" gate="G$1" pin="Q5"/>
-<wire x1="101.6" y1="15.24" x2="111.76" y2="15.24" width="0.1524" layer="91"/>
-<label x="106.68" y="15.24" size="1.016" layer="95" font="vector"/>
+<pinref part="U15" gate="G$1" pin="Q2"/>
+<wire x1="111.76" y1="22.86" x2="101.6" y2="22.86" width="0.1524" layer="91"/>
+<label x="106.68" y="22.86" size="1.016" layer="95" font="vector"/>
 </segment>
 </net>
@@
 </segment>
 <segment>
-<pinref part="U15" gate="G$1" pin="Q4"/>
-<wire x1="111.76" y1="17.78" x2="101.6" y2="17.78" width="0.1524" layer="91"/>
-<label x="106.68" y="17.78" size="1.016" layer="95" font="vector"/>
+<pinref part="U15" gate="G$1" pin="Q3"/>
+<wire x1="101.6" y1="20.32" x2="111.76" y2="20.32" width="0.1524" layer="91"/>
+<label x="106.68" y="20.32" size="1.016" layer="95" font="vector"/>
 </segment>
 </net>
@@
 </segment>
 <segment>
-<pinref part="U15" gate="G$1" pin="Q3"/>
-<wire x1="101.6" y1="20.32" x2="111.76" y2="20.32" width="0.1524" layer="91"/>
-<label x="106.68" y="20.32" size="1.016" layer="95" font="vector"/>
+<pinref part="U15" gate="G$1" pin="Q4"/>
+<wire x1="111.76" y1="17.78" x2="101.6" y2="17.78" width="0.1524" layer="91"/>
+<label x="106.68" y="17.78" size="1.016" layer="95" font="vector"/>
 </segment>
 </net>
@@
 </segment>
 <segment>
-<pinref part="U15" gate="G$1" pin="Q1"/>
-<wire x1="101.6" y1="25.4" x2="111.76" y2="25.4" width="0.1524" layer="91"/>
-<label x="106.68" y="25.4" size="1.016" layer="95" font="vector"/>
+<pinref part="U15" gate="G$1" pin="Q6"/>
+<wire x1="111.76" y1="12.7" x2="101.6" y2="12.7" width="0.1524" layer="91"/>
+<label x="106.68" y="12.7" size="1.016" layer="95" font="vector"/>
 </segment>
 </net>
@@
 </segment>
 <segment>
-<pinref part="U15" gate="G$1" pin="Q0"/>
-<wire x1="101.6" y1="27.94" x2="111.76" y2="27.94" width="0.1524" layer="91"/>
-<label x="106.68" y="27.94" size="1.016" layer="95" font="vector"/>
+<pinref part="U15" gate="G$1" pin="Q7"/>
+<wire x1="101.6" y1="10.16" x2="111.76" y2="10.16" width="0.1524" layer="91"/>
+<label x="106.68" y="10.16" size="1.016" layer="95" font="vector"/>
 </segment>
 </net>
@@
 </segment>
 <segment>
-<pinref part="U15" gate="G$1" pin="Q7"/>
-<wire x1="101.6" y1="10.16" x2="111.76" y2="10.16" width="0.1524" layer="91"/>
-<label x="106.68" y="10.16" size="1.016" layer="95" font="vector"/>
+<pinref part="U15" gate="G$1" pin="Q0"/>
+<wire x1="101.6" y1="27.94" x2="111.76" y2="27.94" width="0.1524" layer="91"/>
+<label x="106.68" y="27.94" size="1.016" layer="95" font="vector"/>
 </segment>
 </net>
@@
 </segment>
 <segment>
-<pinref part="U15" gate="G$1" pin="Q2"/>
-<wire x1="111.76" y1="22.86" x2="101.6" y2="22.86" width="0.1524" layer="91"/>
-<label x="106.68" y="22.86" size="1.016" layer="95" font="vector"/>
+<pinref part="U15" gate="G$1" pin="Q5"/>
+<wire x1="101.6" y1="15.24" x2="111.76" y2="15.24" width="0.1524" layer="91"/>
+<label x="106.68" y="15.24" size="1.016" layer="95" font="vector"/>
 </segment>
 </net>
@@
 </segment>
 <segment>
-<pinref part="U14" gate="G$1" pin="Q7"/>
-<wire x1="101.6" y1="43.18" x2="111.76" y2="43.18" width="0.1524" layer="91"/>
-<label x="106.68" y="43.18" size="1.016" layer="95" font="vector"/>
+<pinref part="U14" gate="G$1" pin="Q1"/>
+<wire x1="101.6" y1="58.42" x2="111.76" y2="58.42" width="0.1524" layer="91"/>
+<label x="106.68" y="58.42" size="1.016" layer="95" font="vector"/>
 </segment>
 </net>
@@
 </segment>
 <segment>
-<pinref part="U14" gate="G$1" pin="Q6"/>
-<wire x1="111.76" y1="45.72" x2="101.6" y2="45.72" width="0.1524" layer="91"/>
-<label x="106.68" y="45.72" size="1.016" layer="95" font="vector"/>
+<pinref part="U14" gate="G$1" pin="Q2"/>
+<wire x1="111.76" y1="55.88" x2="101.6" y2="55.88" width="0.1524" layer="91"/>
+<label x="106.68" y="55.88" size="1.016" layer="95" font="vector"/>
 </segment>
 </net>
@@
 </segment>
 <segment>
-<pinref part="U14" gate="G$1" pin="Q5"/>
-<wire x1="101.6" y1="48.26" x2="111.76" y2="48.26" width="0.1524" layer="91"/>
-<label x="106.68" y="48.26" size="1.016" layer="95" font="vector"/>
+<pinref part="U14" gate="G$1" pin="Q3"/>
+<wire x1="101.6" y1="53.34" x2="111.76" y2="53.34" width="0.1524" layer="91"/>
+<label x="106.68" y="53.34" size="1.016" layer="95" font="vector"/>
 </segment>
 </net>
@@
 </segment>
 <segment>
-<pinref part="U14" gate="G$1" pin="Q3"/>
-<wire x1="101.6" y1="53.34" x2="111.76" y2="53.34" width="0.1524" layer="91"/>
-<label x="106.68" y="53.34" size="1.016" layer="95" font="vector"/>
+<pinref part="U14" gate="G$1" pin="Q5"/>
+<wire x1="101.6" y1="48.26" x2="111.76" y2="48.26" width="0.1524" layer="91"/>
+<label x="106.68" y="48.26" size="1.016" layer="95" font="vector"/>
 </segment>
 </net>
@@
 </segment>
 <segment>
-<pinref part="U14" gate="G$1" pin="Q2"/>
-<wire x1="111.76" y1="55.88" x2="101.6" y2="55.88" width="0.1524" layer="91"/>
-<label x="106.68" y="55.88" size="1.016" layer="95" font="vector"/>
+<pinref part="U14" gate="G$1" pin="Q6"/>
+<wire x1="111.76" y1="45.72" x2="101.6" y2="45.72" width="0.1524" layer="91"/>
+<label x="106.68" y="45.72" size="1.016" layer="95" font="vector"/>
 </segment>
 </net>
@@
 </segment>
 <segment>
-<pinref part="U14" gate="G$1" pin="Q1"/>
-<wire x1="101.6" y1="58.42" x2="111.76" y2="58.42" width="0.1524" layer="91"/>
-<label x="106.68" y="58.42" size="1.016" layer="95" font="vector"/>
+<pinref part="U14" gate="G$1" pin="Q7"/>
+<wire x1="101.6" y1="43.18" x2="111.76" y2="43.18" width="0.1524" layer="91"/>
+<label x="106.68" y="43.18" size="1.016" layer="95" font="vector"/>
 </segment>
 </net>
@@
 <junction x="81.28" y="165.1"/>
 <pinref part="C9" gate="G$1" pin="P$2"/>
-<wire x1="50.8" y1="165.1" x2="55.88" y2="165.1" width="0.1524" layer="91"/>
-<pinref part="R6" gate="G$1" pin="P$1"/>
-<wire x1="55.88" y1="165.1" x2="81.28" y2="165.1" width="0.1524" layer="91"/>
-<wire x1="55.88" y1="170.18" x2="55.88" y2="165.1" width="0.1524" layer="91"/>
-<junction x="55.88" y="165.1"/>
+<wire x1="73.66" y1="165.1" x2="81.28" y2="165.1" width="0.1524" layer="91"/>
 </segment>
 </net>
@@
 <segment>
 <pinref part="C9" gate="G$1" pin="P$1"/>
-<wire x1="30.48" y1="165.1" x2="40.64" y2="165.1" width="0.1524" layer="91"/>
-<label x="30.48" y="165.1" size="1.016" layer="95" font="vector"/>
+<wire x1="53.34" y1="165.1" x2="63.5" y2="165.1" width="0.1524" layer="91"/>
+<label x="53.34" y="165.1" size="1.016" layer="95" font="vector"/>
 </segment>
 </net>

Commit message: Almost done!
Connections:
- removed net P13: U1.P13
- new net 3.3V_SENSE: 3.3V.P$1
- new net P7: U1.P7
- net !RES!_PROP: now also U1.P11; no longer U1.P12
- net !RST!_PIC32: now also U1.P8; no longer U1.P9
- net 3.3V: no longer 3.3V.P$1
- net RX_PIC32: now also U1.P10; no longer U1.P7
- net RX_PROP: now also U1.P13; no longer U1.P10
- net TX_PIC32: now also U1.P9; no longer U1.P8
- net TX_PROP: now also U1.P12; no longer U1.P11
Changed lines of the file:
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@@
 <?xml version="1.0" encoding="utf-8"?>
 <!DOCTYPE eagle SYSTEM "eagle.dtd">
-<eagle version="6.6.0">
+<eagle version="6.5.0">
 <drawing>
 <settings>
@@
 <net name="3.3V" class="0">
 <segment>
-<pinref part="3.3V" gate="G$1" pin="P$1"/>
-<wire x1="-40.64" y1="-101.6" x2="-33.02" y2="-101.6" width="0.1524" layer="91"/>
-<label x="-38.1" y="-101.6" size="1.016" layer="95" font="vector"/>
-</segment>
-<segment>
 <pinref part="R5" gate="G$1" pin="P$2"/>
 <wire x1="81.28" y1="180.34" x2="81.28" y2="182.88" width="0.1524" layer="91"/>
@@
 </segment>
 </net>
-<net name="P13" class="0">
-<segment>
-<pinref part="U1" gate="G$1" pin="P13"/>
-<wire x1="99.06" y1="127" x2="86.36" y2="127" width="0.1524" layer="91"/>
-<label x="86.36" y="127" size="1.016" layer="95" font="vector"/>
-</segment>
-</net>
 <net name="P14" class="0">
 <segment>
@@
 </segment>
 <segment>
-<pinref part="U1" gate="G$1" pin="P10"/>
-<wire x1="86.36" y1="134.62" x2="99.06" y2="134.62" width="0.1524" layer="91"/>
-<label x="86.36" y="134.62" size="1.016" layer="95" font="vector"/>
+<pinref part="U1" gate="G$1" pin="P13"/>
+<wire x1="99.06" y1="127" x2="86.36" y2="127" width="0.1524" layer="91"/>
+<label x="86.36" y="127" size="1.016" layer="95" font="vector"/>
 </segment>
 </net>
@@
 </segment>
 <segment>
-<pinref part="U1" gate="G$1" pin="P11"/>
-<wire x1="99.06" y1="132.08" x2="86.36" y2="132.08" width="0.1524" layer="91"/>
-<label x="86.36" y="132.08" size="1.016" layer="95" font="vector"/>
+<pinref part="U1" gate="G$1" pin="P12"/>
+<wire x1="86.36" y1="129.54" x2="99.06" y2="129.54" width="0.1524" layer="91"/>
+<label x="86.36" y="129.54" size="1.016" layer="95" font="vector"/>
 </segment>
 </net>
@@
 </segment>
 <segment>
-<pinref part="U1" gate="G$1" pin="P12"/>
-<wire x1="86.36" y1="129.54" x2="99.06" y2="129.54" width="0.1524" layer="91"/>
-<label x="86.36" y="129.54" size="1.016" layer="95" font="vector"/>
+<pinref part="U1" gate="G$1" pin="P11"/>
+<wire x1="99.06" y1="132.08" x2="86.36" y2="132.08" width="0.1524" layer="91"/>
+<label x="86.36" y="132.08" size="1.016" layer="95" font="vector"/>
 </segment>
 </net>
@@
 </segment>
 <segment>
-<pinref part="U1" gate="G$1" pin="P7"/>
-<wire x1="99.06" y1="142.24" x2="86.36" y2="142.24" width="0.1524" layer="91"/>
-<label x="86.36" y="142.24" size="1.016" layer="95" font="vector"/>
+<pinref part="U1" gate="G$1" pin="P10"/>
+<wire x1="86.36" y1="134.62" x2="99.06" y2="134.62" width="0.1524" layer="91"/>
+<label x="86.36" y="134.62" size="1.016" layer="95" font="vector"/>
 </segment>
 </net>
@@
 </segment>
 <segment>
-<pinref part="U1" gate="G$1" pin="P8"/>
-<wire x1="86.36" y1="139.7" x2="99.06" y2="139.7" width="0.1524" layer="91"/>
-<label x="86.36" y="139.7" size="1.016" layer="95" font="vector"/>
+<pinref part="U1" gate="G$1" pin="P9"/>
+<wire x1="99.06" y1="137.16" x2="86.36" y2="137.16" width="0.1524" layer="91"/>
+<label x="86.36" y="137.16" size="1.016" layer="95" font="vector"/>
 </segment>
 </net>
@@
 </segment>
 <segment>
-<pinref part="U1" gate="G$1" pin="P9"/>
-<wire x1="99.06" y1="137.16" x2="86.36" y2="137.16" width="0.1524" layer="91"/>
-<label x="86.36" y="137.16" size="1.016" layer="95" font="vector"/>
+<pinref part="U1" gate="G$1" pin="P8"/>
+<wire x1="86.36" y1="139.7" x2="99.06" y2="139.7" width="0.1524" layer="91"/>
+<label x="86.36" y="139.7" size="1.016" layer="95" font="vector"/>
 </segment>
 </net>
@@
 </segment>
 </net>
+<net name="3.3V_SENSE" class="0">
+<segment>
+<pinref part="3.3V" gate="G$1" pin="P$1"/>
+<wire x1="-40.64" y1="-101.6" x2="-33.02" y2="-101.6" width="0.1524" layer="91"/>
+<label x="-38.1" y="-101.6" size="1.016" layer="95" font="vector"/>
+</segment>
+</net>
+<net name="P7" class="0">
+<segment>
+<pinref part="U1" gate="G$1" pin="P7"/>
+<wire x1="99.06" y1="142.24" x2="86.36" y2="142.24" width="0.1524" layer="91"/>
+<label x="86.36" y="142.24" size="1.016" layer="95" font="vector"/>
+</segment>
+</net>

Commit message: routing almost done.
Connections:
- removed net P16: U1.P16
- removed net P17: U1.P17
- removed net P18: U1.P18
- removed net P19: U1.P19
- removed net P20: U1.P20
- removed net P21: U1.P21
- new net P1: U1.P1
- new net P2: U1.P2
- new net P3: U1.P3
- new net P4: U1.P4
- new net P5: U1.P5
- new net P6: U1.P6
- net 165_CLK: now also U1.P16; no longer U1.P4
- net 165_DATA: now also U1.P18; no longer U1.P6
- net 165_LOAD: now also U1.P17; no longer U1.P5
- net 595_CLK: now also U1.P19; no longer U1.P1
- net 595_DATA: now also U1.P21; no longer U1.P3
- net 595_LAT: now also U1.P20; no longer U1.P2
Changed lines of the file:
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@@
 <?xml version="1.0" encoding="utf-8"?>
 <!DOCTYPE eagle SYSTEM "eagle.dtd">
-<eagle version="6.5.0">
+<eagle version="6.6.0">
 <drawing>
 <settings>
@@
 </segment>
 </net>
-<net name="P16" class="0">
-<segment>
-<pinref part="U1" gate="G$1" pin="P16"/>
-<wire x1="119.38" y1="121.92" x2="132.08" y2="121.92" width="0.1524" layer="91"/>
-<label x="121.92" y="121.92" size="1.016" layer="95" font="vector"/>
-</segment>
-</net>
-<net name="P17" class="0">
-<segment>
-<pinref part="U1" gate="G$1" pin="P17"/>
-<wire x1="132.08" y1="124.46" x2="119.38" y2="124.46" width="0.1524" layer="91"/>
-<label x="121.92" y="124.46" size="1.016" layer="95" font="vector"/>
-</segment>
-</net>
 <net name="P27" class="0">
 <segment>
@@
 </segment>
 </net>
-<net name="P21" class="0">
-<segment>
-<pinref part="U1" gate="G$1" pin="P21"/>
-<wire x1="132.08" y1="134.62" x2="119.38" y2="134.62" width="0.1524" layer="91"/>
-<label x="121.92" y="134.62" size="1.016" layer="95" font="vector"/>
-</segment>
-</net>
-<net name="P20" class="0">
-<segment>
-<pinref part="U1" gate="G$1" pin="P20"/>
-<wire x1="119.38" y1="132.08" x2="132.08" y2="132.08" width="0.1524" layer="91"/>
-<label x="121.92" y="132.08" size="1.016" layer="95" font="vector"/>
-</segment>
-</net>
 <net name="SCL" class="0">
 <segment>
@@
 </segment>
 </net>
-<net name="P18" class="0">
-<segment>
-<pinref part="U1" gate="G$1" pin="P18"/>
-<wire x1="119.38" y1="127" x2="132.08" y2="127" width="0.1524" layer="91"/>
-<label x="121.92" y="127" size="1.016" layer="95" font="vector"/>
-</segment>
-</net>
 <net name="V_USB_0" class="0">
 <segment>
@@
 </segment>
 </net>
-<net name="P19" class="0">
-<segment>
-<pinref part="U1" gate="G$1" pin="P19"/>
-<wire x1="132.08" y1="129.54" x2="119.38" y2="129.54" width="0.1524" layer="91"/>
-<label x="121.92" y="129.54" size="1.016" layer="95" font="vector"/>
-</segment>
-</net>
 <net name="N$32" class="0">
 <segment>
@@
 </segment>
 <segment>
-<pinref part="U1" gate="G$1" pin="P3"/>
-<wire x1="99.06" y1="152.4" x2="86.36" y2="152.4" width="0.1524" layer="91"/>
-<label x="86.36" y="152.4" size="1.016" layer="95" font="vector"/>
+<pinref part="U1" gate="G$1" pin="P21"/>
+<wire x1="132.08" y1="134.62" x2="119.38" y2="134.62" width="0.1524" layer="91"/>
+<label x="121.92" y="134.62" size="1.016" layer="95" font="vector"/>
 </segment>
 </net>
@@
 </segment>
 <segment>
-<pinref part="U1" gate="G$1" pin="P1"/>
-<wire x1="99.06" y1="157.48" x2="86.36" y2="157.48" width="0.1524" layer="91"/>
-<label x="86.36" y="157.48" size="1.016" layer="95" font="vector"/>
+<pinref part="U1" gate="G$1" pin="P19"/>
+<wire x1="132.08" y1="129.54" x2="119.38" y2="129.54" width="0.1524" layer="91"/>
+<label x="121.92" y="129.54" size="1.016" layer="95" font="vector"/>
 </segment>
 </net>
@@
 </segment>
 <segment>
-<pinref part="U1" gate="G$1" pin="P2"/>
-<wire x1="86.36" y1="154.94" x2="99.06" y2="154.94" width="0.1524" layer="91"/>
-<label x="86.36" y="154.94" size="1.016" layer="95" font="vector"/>
+<pinref part="U1" gate="G$1" pin="P20"/>
+<wire x1="119.38" y1="132.08" x2="132.08" y2="132.08" width="0.1524" layer="91"/>
+<label x="121.92" y="132.08" size="1.016" layer="95" font="vector"/>
 </segment>
 </net>
@@
 </segment>
 <segment>
-<pinref part="U1" gate="G$1" pin="P6"/>
-<wire x1="86.36" y1="144.78" x2="99.06" y2="144.78" width="0.1524" layer="91"/>
-<label x="86.36" y="144.78" size="1.016" layer="95" font="vector"/>
+<pinref part="U1" gate="G$1" pin="P18"/>
+<wire x1="119.38" y1="127" x2="132.08" y2="127" width="0.1524" layer="91"/>
+<label x="121.92" y="127" size="1.016" layer="95" font="vector"/>
 </segment>
 </net>
@@
 </segment>
 <segment>
-<pinref part="U1" gate="G$1" pin="P4"/>
-<wire x1="86.36" y1="149.86" x2="99.06" y2="149.86" width="0.1524" layer="91"/>
-<label x="86.36" y="149.86" size="1.016" layer="95" font="vector"/>
+<pinref part="U1" gate="G$1" pin="P16"/>
+<wire x1="119.38" y1="121.92" x2="132.08" y2="121.92" width="0.1524" layer="91"/>
+<label x="121.92" y="121.92" size="1.016" layer="95" font="vector"/>
 </segment>
 </net>
@@
 </segment>
 <segment>
-<pinref part="U1" gate="G$1" pin="P5"/>
-<wire x1="99.06" y1="147.32" x2="86.36" y2="147.32" width="0.1524" layer="91"/>
-<label x="86.36" y="147.32" size="1.016" layer="95" font="vector"/>
+<pinref part="U1" gate="G$1" pin="P17"/>
+<wire x1="132.08" y1="124.46" x2="119.38" y2="124.46" width="0.1524" layer="91"/>
+<label x="121.92" y="124.46" size="1.016" layer="95" font="vector"/>
 </segment>
 </net>
@@
 </segment>
 </net>
+<net name="P4" class="0">
+<segment>
+<pinref part="U1" gate="G$1" pin="P4"/>
+<wire x1="86.36" y1="149.86" x2="99.06" y2="149.86" width="0.1524" layer="91"/>
+<label x="86.36" y="149.86" size="1.016" layer="95" font="vector"/>
+</segment>
+</net>
+<net name="P5" class="0">
+<segment>
+<pinref part="U1" gate="G$1" pin="P5"/>
+<wire x1="99.06" y1="147.32" x2="86.36" y2="147.32" width="0.1524" layer="91"/>
+<label x="86.36" y="147.32" size="1.016" layer="95" font="vector"/>
+</segment>
+</net>
+<net name="P6" class="0">
+<segment>
+<pinref part="U1" gate="G$1" pin="P6"/>
+<wire x1="86.36" y1="144.78" x2="99.06" y2="144.78" width="0.1524" layer="91"/>
+<label x="86.36" y="144.78" size="1.016" layer="95" font="vector"/>
+</segment>
+</net>
+<net name="P1" class="0">
+<segment>
+<pinref part="U1" gate="G$1" pin="P1"/>
+<wire x1="99.06" y1="157.48" x2="86.36" y2="157.48" width="0.1524" layer="91"/>
+<label x="86.36" y="157.48" size="1.016" layer="95" font="vector"/>
+</segment>
+</net>
+<net name="P2" class="0">
+<segment>
+<pinref part="U1" gate="G$1" pin="P2"/>
+<wire x1="86.36" y1="154.94" x2="99.06" y2="154.94" width="0.1524" layer="91"/>
+<label x="86.36" y="154.94" size="1.016" layer="95" font="vector"/>
+</segment>
+</net>
+<net name="P3" class="0">
+<segment>
+<pinref part="U1" gate="G$1" pin="P3"/>
+<wire x1="99.06" y1="152.4" x2="86.36" y2="152.4" width="0.1524" layer="91"/>
+<label x="86.36" y="152.4" size="1.016" layer="95" font="vector"/>
+</segment>
+</net>

Commit message: Almost done.
Need to change drill size.
Parts:
- added C26, C27, C28, C29, C30, C31, C32, C33, C34, C35, C36, C37, C38, C39: 0.1uF, MF_Passives:CAPACITOR_NP_0603
- !RES!_PROP, !RST!_PIC32, 12V, 3.3V, 50V, 5V, BACK_OUT, COIN_OUT, DMD_1, DMD_11, DMD_13, DMD_3, DMD_5, DMD_7, DMD_9, DOOR_OUT, ENTER_OUT, EXT_RGB_CLK, EXT_RGB_DATA, GI_R_0, GI_R_1, GI_R_10, GI_R_11, GI_R_12, GI_R_13, GI_R_14, GI_R_15, GI_R_2, GI_R_3, GI_R_4, GI_R_5, GI_R_6, GI_R_7, GI_R_8, GI_R_9, GND, LIGHT_C_0, LIGHT_C_1, LIGHT_C_2, LIGHT_C_3, LIGHT_C_4, LIGHT_C_5, LIGHT_C_6, LIGHT_C_7, LIGHT_R_0, LIGHT_R_1, LIGHT_R_2, LIGHT_R_3, LIGHT_R_4, LIGHT_R_5, LIGHT_R_6, LIGHT_R_7, L_FLIP_OUT, OPTO_1_, OPTO_2_, OPTO_3_, OPTO_4_, OPTO_5_, OPTO_6_, OPTO_7_, PROP_AUX0, PROP_AUX1, RGB_BOUT_L, RGB_BOUT_R, RGB_GOUT_L, RGB_GOUT_R, RGB_ROUT_L, RGB_ROUT_R, RX_PIC32, RX_PROP, R_FLIP_OUT, SD_CS, SD_DI, SD_DO, SD_SCLK, SERVO_0_, SERVO_1_, SERVO_2_, SERVO_3_, SERVO_4_, SOL_GND, SOL_PWR_0, SOL_PWR_1, SOL_PWR_10, SOL_PWR_11, SOL_PWR_12, SOL_PWR_13, SOL_PWR_14, SOL_PWR_15, SOL_PWR_16, SOL_PWR_17, SOL_PWR_18, SOL_PWR_19, SOL_PWR_2, SOL_PWR_20, SOL_PWR_21, SOL_PWR_22, SOL_PWR_23, SOL_PWR_3, SOL_PWR_4, SOL_PWR_5, SOL_PWR_6, SOL_PWR_7, SOL_PWR_8, SOL_PWR_9, ST_BU_OUT, ST_LI_, SW_C_0, SW_C_1, SW_C_2, SW_C_3, SW_C_4, SW_C_5, SW_C_6, SW_C_7, SW_R_0, SW_R_1, SW_R_2, SW_R_3, SW_R_4, SW_R_5, SW_R_6, SW_R_7, S_L, S_R, TILT_OUT, TX_PIC32, TX_PROP, USER_0_OUT: value (none) -> 0914-3-15-20-77-14-11-0
Connections:
- net 3.3V: now also C26.P$1, C27.P$1, C28.P$1, C29.P$1, C30.P$1, C31.P$1, C32.P$1, C33.P$1, C34.P$1, C35.P$1, C36.P$1, C37.P$1, C38.P$1, C39.P$1
- net 3.3V_SENSE: now also U9.A_2
- net GND: now also C26.P$2, C27.P$2, C28.P$2, C29.P$2, C30.P$2, C31.P$2, C32.P$2, C33.P$2, C34.P$2, C35.P$2, C36.P$2, C37.P$2, C38.P$2, C39.P$2
Other:
- moved on the sheet: 12V, 5V, BACK_OUT, COIN_OUT, DMD_1, DMD_11, DMD_13, DMD_3, DMD_5, DMD_7, DMD_9, DOOR_OUT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
