File: Hardware/Pinheck Test Jig/PinHeck Test Jig.sch (EAGLE design)
At the start: 327 parts, among them U1 P8X32A-Q44, U10 BSO080P03NS3E G, U11 BSO080P03NS3E G, U12 MF-DSC-SOT233-MMBT3904, U13 MF-DSC-SOT233-MMBT3904, U14 CD74HC595M96, U15 CD74HC595M96, U16 CD74HC165M96, U17 CD74HC165M96, U18 CD74HC165M96, U19 CD74HC165M96, U2 CAT24C512WI-GT3, U20 CD74HC165M96, U21 CD74HC165M96, U22 CD74HC165M96, U23 CD74HC165M96, U24 CD74HC165M96, U26 CD74HC165M96, U27 CD74HC165M96, U28 CD74HC165M96, U29 CD74HC165M96, U3 FT230XS, U30 CD74HC165M96, U4 IP4234CZ6, U5 NCP1117DT33G, U6 NCP1117DT50G, U7 INA139NA/3K, U8 INA139NA/3K, U9 MAX11613EUA+, X1 ABMM-6.000MHZ-B2-T

Commit message: Test Jig done.
Parts:
- added H18, H19, H20, H21: 2263-2, PP_Connectors:MOUNT_HOLE120MIL
- H1, H10, H11, H12, H13, H14, H15, H16, H17, H2, H3, H4, H5, H6, H7, H8, H9: value MOUNT_HOLE150MIL -> 2263-2; device PP_Connectors:MOUNT_HOLE150MIL -> PP_Connectors:MOUNT_HOLE120MIL
Changed lines of the file:
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@@
 <?xml version="1.0" encoding="utf-8"?>
 <!DOCTYPE eagle SYSTEM "eagle.dtd">
-<eagle version="6.5.0">
+<eagle version="6.6.0">
 <drawing>
 <settings>
@@
 </classes>
 <parts>
-<part name="H2" library="PP_Connectors" deviceset="MOUNT_HOLE" device="150MIL"/>
-<part name="H4" library="PP_Connectors" deviceset="MOUNT_HOLE" device="150MIL"/>
-<part name="H6" library="PP_Connectors" deviceset="MOUNT_HOLE" device="150MIL"/>
-<part name="H8" library="PP_Connectors" deviceset="MOUNT_HOLE" device="150MIL"/>
-<part name="H10" library="PP_Connectors" deviceset="MOUNT_HOLE" device="150MIL"/>
-<part name="H12" library="PP_Connectors" deviceset="MOUNT_HOLE" device="150MIL"/>
-<part name="H1" library="PP_Connectors" deviceset="MOUNT_HOLE" device="150MIL"/>
-<part name="H3" library="PP_Connectors" deviceset="MOUNT_HOLE" device="150MIL"/>
-<part name="H5" library="PP_Connectors" deviceset="MOUNT_HOLE" device="150MIL"/>
-<part name="H7" library="PP_Connectors" deviceset="MOUNT_HOLE" device="150MIL"/>
-<part name="H9" library="PP_Connectors" deviceset="MOUNT_HOLE" device="150MIL"/>
-<part name="H11" library="PP_Connectors" deviceset="MOUNT_HOLE" device="150MIL"/>
-<part name="H13" library="PP_Connectors" deviceset="MOUNT_HOLE" device="150MIL"/>
-<part name="H14" library="PP_Connectors" deviceset="MOUNT_HOLE" device="150MIL"/>
-<part name="H15" library="PP_Connectors" deviceset="MOUNT_HOLE" device="150MIL"/>
-<part name="H17" library="PP_Connectors" deviceset="MOUNT_HOLE" device="150MIL"/>
-<part name="H16" library="PP_Connectors" deviceset="MOUNT_HOLE" device="150MIL"/>
+<part name="H2" library="PP_Connectors" deviceset="MOUNT_HOLE" device="120MIL" value="2263-2"/>
+<part name="H4" library="PP_Connectors" deviceset="MOUNT_HOLE" device="120MIL" value="2263-2"/>
+<part name="H6" library="PP_Connectors" deviceset="MOUNT_HOLE" device="120MIL" value="2263-2"/>
+<part name="H8" library="PP_Connectors" deviceset="MOUNT_HOLE" device="120MIL" value="2263-2"/>
+<part name="H10" library="PP_Connectors" deviceset="MOUNT_HOLE" device="120MIL" value="2263-2"/>
+<part name="H12" library="PP_Connectors" deviceset="MOUNT_HOLE" device="120MIL" value="2263-2"/>
+<part name="H1" library="PP_Connectors" deviceset="MOUNT_HOLE" device="120MIL" value="2263-2"/>
+<part name="H3" library="PP_Connectors" deviceset="MOUNT_HOLE" device="120MIL" value="2263-2"/>
+<part name="H5" library="PP_Connectors" deviceset="MOUNT_HOLE" device="120MIL" value="2263-2"/>
+<part name="H7" library="PP_Connectors" deviceset="MOUNT_HOLE" device="120MIL" value="2263-2"/>
+<part name="H9" library="PP_Connectors" deviceset="MOUNT_HOLE" device="120MIL" value="2263-2"/>
+<part name="H11" library="PP_Connectors" deviceset="MOUNT_HOLE" device="120MIL" value="2263-2"/>
+<part name="H13" library="PP_Connectors" deviceset="MOUNT_HOLE" device="120MIL" value="2263-2"/>
+<part name="H14" library="PP_Connectors" deviceset="MOUNT_HOLE" device="120MIL" value="2263-2"/>
+<part name="H15" library="PP_Connectors" deviceset="MOUNT_HOLE" device="120MIL" value="2263-2"/>
+<part name="H17" library="PP_Connectors" deviceset="MOUNT_HOLE" device="120MIL" value="2263-2"/>
+<part name="H16" library="PP_Connectors" deviceset="MOUNT_HOLE" device="120MIL" value="2263-2"/>
 <part name="SW_R_7" library="PP_Connectors" deviceset="POGO_PIN" device="_0914-3-15-20-77-14-11-0" value="0914-3-15-20-77-14-11-0"/>
 <part name="SW_R_6" library="PP_Connectors" deviceset="POGO_PIN" device="_0914-3-15-20-77-14-11-0" value="0914-3-15-20-77-14-11-0"/>
@@
 <part name="C38" library="MF_Passives" deviceset="CAPACITOR_NP" device="_0603" value="0.1uF"/>
 <part name="C39" library="MF_Passives" deviceset="CAPACITOR_NP" device="_0603" value="0.1uF"/>
+<part name="H18" library="PP_Connectors" deviceset="MOUNT_HOLE" device="120MIL" value="2263-2"/>
+<part name="H19" library="PP_Connectors" deviceset="MOUNT_HOLE" device="120MIL" value="2263-2"/>
+<part name="H20" library="PP_Connectors" deviceset="MOUNT_HOLE" device="120MIL" value="2263-2"/>
+<part name="H21" library="PP_Connectors" deviceset="MOUNT_HOLE" device="120MIL" value="2263-2"/>
 </parts>
 <sheets>
@@
 <instance part="C38" gate="G$1" x="276.86" y="-436.88"/>
 <instance part="C39" gate="G$1" x="287.02" y="-436.88"/>
+<instance part="H18" gate="G$1" x="-2.54" y="-30.48"/>
+<instance part="H19" gate="G$1" x="-15.24" y="-38.1"/>
+<instance part="H20" gate="G$1" x="-2.54" y="-38.1"/>
+<instance part="H21" gate="G$1" x="-15.24" y="-45.72"/>
 </instances>
 <busses>
