File: Hardware/Spooky Sound System/Spooky Sound System.sch (EAGLE design)
At the start: 85 parts, among them J1 SJ1-3533NS, J2 1546215-2, J3 1546215-2, J4 1546215-2, J5 1546215-2, U1 TDA7387, U2 AZ4558C, U3 AZ4558C, U4 AZ4558C, U5 AZ4558C, U6 AZ4558C

Commit message: Initial routing done.
Parts:
- J2: LABEL01 L+ -> L-; LABEL02 L- -> L+
- J3: LABEL01 R+ -> R-; LABEL02 R- -> R+
Connections:
- net L+: now also J2.PIN2; no longer J2.PIN1
- net L-: now also J2.PIN1; no longer J2.PIN2
- net R+: now also J3.PIN2; no longer J3.PIN1
- net R-: now also J3.PIN1; no longer J3.PIN2
Other:
- moved on the sheet: J2, J3
Changed lines of the file:
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@@
 <part name="U$16" library="MF_Aesthetics" deviceset="GND_RAIL" device="" value="GND"/>
 <part name="J2" library="PP_Connectors" deviceset="CON_01X02" device="_1546215-2" value="1546215-2">
-<attribute name="LABEL01" value="L+"/>
-<attribute name="LABEL02" value="L-"/>
+<attribute name="LABEL01" value="L-"/>
+<attribute name="LABEL02" value="L+"/>
 </part>
 <part name="J3" library="PP_Connectors" deviceset="CON_01X02" device="_1546215-2" value="1546215-2">
-<attribute name="LABEL01" value="R+"/>
-<attribute name="LABEL02" value="R-"/>
+<attribute name="LABEL01" value="R-"/>
+<attribute name="LABEL02" value="R+"/>
 </part>
 <part name="J4" library="PP_Connectors" deviceset="CON_01X02" device="_1546215-2" value="1546215-2">
@@
 <instance part="J1" gate="G$1" x="-279.4" y="218.44" rot="MR180"/>
 <instance part="U$16" gate="G$1" x="-264.16" y="208.28"/>
-<instance part="J2" gate="G$1" x="30.48" y="190.5"/>
-<instance part="J3" gate="G$1" x="30.48" y="172.72"/>
+<instance part="J2" gate="G$1" x="30.48" y="187.96" rot="MR180"/>
+<instance part="J3" gate="G$1" x="30.48" y="170.18" rot="MR180"/>
 <instance part="J4" gate="G$1" x="30.48" y="154.94"/>
 <instance part="J5" gate="G$1" x="-271.78" y="236.22" rot="MR0"/>
@@
 <wire x1="5.08" y1="190.5" x2="27.94" y2="190.5" width="0.1524" layer="91"/>
 <label x="15.24" y="190.5" size="1.016" layer="95" font="vector"/>
-<pinref part="J2" gate="G$1" pin="PIN1"/>
+<pinref part="J2" gate="G$1" pin="PIN2"/>
 </segment>
 </net>
@@
 <label x="15.24" y="185.42" size="1.016" layer="95" font="vector"/>
 <wire x1="20.32" y1="185.42" x2="20.32" y2="187.96" width="0.1524" layer="91"/>
-<pinref part="J2" gate="G$1" pin="PIN2"/>
+<pinref part="J2" gate="G$1" pin="PIN1"/>
 <wire x1="20.32" y1="187.96" x2="27.94" y2="187.96" width="0.1524" layer="91"/>
 </segment>
@@
 <wire x1="5.08" y1="172.72" x2="27.94" y2="172.72" width="0.1524" layer="91"/>
 <label x="15.24" y="172.72" size="1.016" layer="95" font="vector"/>
-<pinref part="J3" gate="G$1" pin="PIN1"/>
+<pinref part="J3" gate="G$1" pin="PIN2"/>
 </segment>
 </net>
@@
 <label x="15.24" y="167.64" size="1.016" layer="95" font="vector"/>
 <wire x1="20.32" y1="167.64" x2="20.32" y2="170.18" width="0.1524" layer="91"/>
-<pinref part="J3" gate="G$1" pin="PIN2"/>
-<wire x1="20.32" y1="170.18" x2="27.94" y2="170.18" width="0.1524" layer="91"/>
-</segment>
-</net>
+<pinref part="J3" gate="G$1" pin="PIN1"/>
+<wire x1="27.94" y1="170.18" x2="20.32" y2="170.18" width="0.1524" layer="91"/>
+</segment>
+</net>

Commit message: Finished routing
Just needs tweaking and final look over.
Parts:
- removed HI, LOW: 100K, PP_Passives:DUAL_TAPER_POTENTIOMETER
- removed J1: SJ1-3533NS, PP_Connectors:TRS_SHIELD_JACK_SJ1-3533NS
- added AUDINPUT: SJ1-3533NS, PP_Connectors:TRS_SHIELD_JACK_SJ1-3533NS
- added BASS, TREBEL: 100K, PP_Passives:DUAL_TAPER_POTENTIOMETER
- added H1, H2, H3, H4: MOUNT_HOLE150MIL, PP_Connectors:MOUNT_HOLE150MIL
- added LOGO1: SPOOKY_LOGOSPOOKY_LOGO, PP_Aesthetics:SPOOKY_LOGOSPOOKY_LOGO
- added U$17: LHE_FRAME, PP_Aesthetics:LHE_FRAME
- added U$18: LHE_LOGOLHE_LOGO, PP_Aesthetics:LHE_LOGOLHE_LOGO
- added U$19: MF_LOGOLOGO_TEXT, PP_Aesthetics:MF_LOGOLOGO_TEXT
Connections:
- net AUD_IN_L: now also AUDINPUT.T; no longer J1.T
- net AUD_IN_R: now also AUDINPUT.R; no longer J1.R
- net GND: now also AUDINPUT.S, AUDINPUT.SHIELD; no longer J1.S, J1.SHIELD
- net N$14: now also TREBEL_B.1; no longer HI_B.1
- net N$15: now also TREBEL_B.2; no longer HI_B.2
- net N$16: now also TREBEL_B.3; no longer HI_B.3
- net N$18: now also BASS_B.2; no longer LOW_B.2
- net N$19: now also BASS_B.1; no longer LOW_B.1
- net N$20: now also BASS_B.3; no longer LOW_B.3
- net N$3: now also TREBEL_A.1; no longer HI_A.1
- net N$4: now also TREBEL_A.2; no longer HI_A.2
- net N$5: now also TREBEL_A.3; no longer HI_A.3
- net N$7: now also BASS_A.2; no longer LOW_A.2
- net N$8: now also BASS_A.1; no longer LOW_A.1
- net N$9: now also BASS_A.3; no longer LOW_A.3
Other:
- moved on the sheet: C1, C10, C11, C12, C13, C14, C15, C16, C17, C18, C19, C2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
