File: Hardware/RPI3_LVDS/RPI3_LVDS.sch (EAGLE design)
At the start: 37 parts, among them J2 87832-6422, J3 1775470-6, U1 DS90C365A, U2 LM1085ISX-5.0/NOPB, U3 ADP3338AKCZ-3.3-RL

Commit message: Uploading camfiles and manufacturing data.
Parts:
- U$14: REVNUM REV: 1 -> REV: 2
Changed lines of the file:
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@@
 <part name="U$14" library="PP_Aesthetics" deviceset="LHE_FRAME" device="">
 <attribute name="DNAME" value="Parker Dillmann"/>
-<attribute name="REVNUM" value="REV: 1"/>
+<attribute name="REVNUM" value="REV: 2"/>
 </part>
 <part name="LOGO1" library="PP_Aesthetics" deviceset="SPOOKY_LOGO" device="SPOOKY_LOGO"/>

Commit message: Fixed LM1085
Parts:
- U$14: REVNUM REV: 2 -> REV: 3
Changed lines of the file:
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@@
 <part name="U$14" library="PP_Aesthetics" deviceset="LHE_FRAME" device="">
 <attribute name="DNAME" value="Parker Dillmann"/>
-<attribute name="REVNUM" value="REV: 2"/>
+<attribute name="REVNUM" value="REV: 3"/>
 </part>
 <part name="LOGO1" library="PP_Aesthetics" deviceset="SPOOKY_LOGO" device="SPOOKY_LOGO"/>
